File: Boards/Audio board rev.a/Audio board rev.a.kicad_sch (KiCad schematic)
At the start: 104 parts, among them J1 CEC card edge connector large, U1 6821, U10 LM324, U11 MC1458, U2 LM339, U3 LM339, U4 ULN2003A, U5 DAC-08, U6 DAC-08, U7 AH5012, U9 LM324

Commit message: more footprints
Parts:
- C1, C2, C21, C24, C3: footprint (none) -> Evan's parts:CP_Radial_Tantal_D4mm_P3.81mm
- C36, C37: footprint (none) -> Capacitor_THT:C_Disc_D3.0mm_W1.6mm_P2.50mm
Changed lines of the file:
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@@
       (effects (font (size 1.27 1.27)) (justify left))
     )
-    (property "Footprint" "" (at 469.5952 276.225 0)
+    (property "Footprint" "Evan's parts:CP_Radial_Tantal_D4mm_P3.81mm" (at 469.5952 276.225 0)
       (effects (font (size 1.27 1.27)) hide)
     )
@@
       (effects (font (size 1.27 1.27)) (justify left))
     )
-    (property "Footprint" "" (at 166.7002 266.7 0)
+    (property "Footprint" "Evan's parts:CP_Radial_Tantal_D4mm_P3.81mm" (at 166.7002 266.7 0)
       (effects (font (size 1.27 1.27)) hide)
     )
@@
       (effects (font (size 1.27 1.27)) (justify left))
     )
-    (property "Footprint" "" (at 489.2802 274.32 0)
+    (property "Footprint" "Evan's parts:CP_Radial_Tantal_D4mm_P3.81mm" (at 489.2802 274.32 0)
       (effects (font (size 1.27 1.27)) hide)
     )
@@
       (effects (font (size 1.27 1.27)) (justify left))
     )
-    (property "Footprint" "" (at 454.9902 276.225 0)
+    (property "Footprint" "Evan's parts:CP_Radial_Tantal_D4mm_P3.81mm" (at 454.9902 276.225 0)
       (effects (font (size 1.27 1.27)) hide)
     )
@@
       (effects (font (size 1.27 1.27)) (justify right))
     )
-    (property "Footprint" "" (at 142.5702 354.33 0)
+    (property "Footprint" "Capacitor_THT:C_Disc_D3.0mm_W1.6mm_P2.50mm" (at 142.5702 354.33 0)
       (effects (font (size 1.27 1.27)) hide)
     )
@@
       (effects (font (size 1.27 1.27)) (justify right))
     )
-    (property "Footprint" "" (at 138.1252 254.635 0)
+    (property "Footprint" "Capacitor_THT:C_Disc_D3.0mm_W1.6mm_P2.50mm" (at 138.1252 254.635 0)
       (effects (font (size 1.27 1.27)) hide)
     )
@@
       (effects (font (size 1.27 1.27)) (justify right))
     )
-    (property "Footprint" "" (at 167.9448 366.395 0)
+    (property "Footprint" "Evan's parts:CP_Radial_Tantal_D4mm_P3.81mm" (at 167.9448 366.395 0)
       (effects (font (size 1.27 1.27)) hide)
     )
