File: Boards/Character board rev.a/Character board rev.a.kicad_pcb (KiCad board)
At the start: 2 copper layers, 184.3 x 186.8 mm, 64 parts, among them J1 card edge, J2 Conn_02x13_Odd_Even, Q1 2N6125, U1 R_Pack07, U10 Unused DIP, U11 ULN2003A, U12 ULN2003A, U13 7406, U14 74LS42, U15 LM741, U16 AH5012, U2 R_Pack07, U3 Unused DIP, U4 Unused DIP, U5 Unused DIP, U6 Board ID header, U7 6821, U8 3.3K, U9 LM741

Commit message: character card rev a done
Parts:
- removed D1: 1N4001, Diode_THT:D_DO-41_SOD81_P12.70mm_Horizontal
- added CR1: 1N4001, Diode_THT:D_DO-41_SOD81_P12.70mm_Horizontal, F.Cu at (174.0, 104.1)
- DS1, DS10, DS11, DS12, DS13, DS14, DS2, DS3, DS4, DS5, DS6, DS7, DS8, DS9: footprint LED_THT:LED_D5.0mm_Horizontal_O3.81mm_Z15.0mm -> Evan's parts:LED_D5.0mm_Horizontal_O3.81mm_Z15.0mm reversed
- J2: value Conn_02x13_Odd_Even -> character connector
- R10: value 47.5KK -> 47.5K
- R7: value ? -> 120
- TP2: value GND -> +5
- TP3: value GND -> +12
- TP4: value GND -> -12
- TP5: value GND -> 24
- U1, U2: value R_Pack07 -> 2.2K
- moved U3 267.0 mm to (106.7, 162.6), turned to 90 degrees
- moved U10 256.1 mm to (137.2, 162.6), turned to 90 degrees
- moved U4 248.6 mm to (106.7, 144.8), turned to 90 degrees
- moved R1 248.5 mm to (127.0, 96.5)
- moved U11 237.5 mm to (137.2, 144.8), turned to 90 degrees
- moved C3 236.5 mm to (176.5, 47.0), turned to 90 degrees
- moved U5 230.1 mm to (106.0, 127.0), turned to 90 degrees
- moved U13 226.6 mm to (137.2, 109.2), turned to 90 degrees
- moved C2 222.9 mm to (172.1, 87.6), turned to 90 degrees
- moved C4 220.1 mm to (156.8, 47.0), turned to 90 degrees
- moved U12 219.2 mm to (137.2, 127.0), turned to 90 degrees
- moved U9 219.1 mm to (104.1, 26.7), turned to 90 degrees
- moved J2 216.4 mm to (173.4, 120.7)
- moved C1 216.0 mm to (165.7, 114.9), turned to -90 degrees
- moved U6 207.1 mm to (106.7, 109.2), turned to 90 degrees
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Connections:
- C10 pad 1: unconnected-(C10-Pad1) -> 5V
- C10 pad 2: unconnected-(C10-Pad2) -> GND
- C11 pad 1: unconnected-(C11-Pad1) -> Net-(C11-Pad1)
- C11 pad 2: unconnected-(C11-Pad2) -> GND
- C5 pad 1: unconnected-(C5-Pad1) -> 24R
- C5 pad 2: unconnected-(C5-Pad2) -> Net-(Q1-C)
- C9 pad 1: unconnected-(C9-Pad1) -> 5V
- C9 pad 2: unconnected-(C9-Pad2) -> GND
- DS1 pad 1: unconnected-(DS1-K-Pad1) -> A0out
- DS1 pad 2: unconnected-(DS1-A-Pad2) -> Net-(DS1-A)
- DS10 pad 1: unconnected-(DS10-K-Pad1) -> B1out
- DS10 pad 2: unconnected-(DS10-A-Pad2) -> Net-(DS10-A)
- DS11 pad 1: unconnected-(DS11-K-Pad1) -> B2out
- DS11 pad 2: unconnected-(DS11-A-Pad2) -> Net-(DS11-A)
- DS12 pad 1: unconnected-(DS12-K-Pad1) -> B3out
- DS12 pad 2: unconnected-(DS12-A-Pad2) -> Net-(DS12-A)
- DS13 pad 1: unconnected-(DS13-K-Pad1) -> B4out
- DS13 pad 2: unconnected-(DS13-A-Pad2) -> Net-(DS13-A)
- DS14 pad 1: unconnected-(DS14-K-Pad1) -> B5out
- DS14 pad 2: unconnected-(DS14-A-Pad2) -> Net-(DS14-A)
- DS2 pad 1: unconnected-(DS2-K-Pad1) -> A1out
- DS2 pad 2: unconnected-(DS2-A-Pad2) -> Net-(DS2-A)
- DS3 pad 1: unconnected-(DS3-K-Pad1) -> A2out
- DS3 pad 2: unconnected-(DS3-A-Pad2) -> Net-(DS3-A)
- DS4 pad 1: unconnected-(DS4-K-Pad1) -> A3out
- DS4 pad 2: unconnected-(DS4-A-Pad2) -> Net-(DS4-A)
- DS5 pad 1: unconnected-(DS5-K-Pad1) -> A4out
- DS5 pad 2: unconnected-(DS5-A-Pad2) -> Net-(DS5-A)
- DS6 pad 1: unconnected-(DS6-K-Pad1) -> A5out
- DS6 pad 2: unconnected-(DS6-A-Pad2) -> Net-(DS6-A)
- DS7 pad 1: unconnected-(DS7-K-Pad1) -> A6out
- DS7 pad 2: unconnected-(DS7-A-Pad2) -> Net-(DS7-A)
- DS8 pad 1: unconnected-(DS8-K-Pad1) -> A7out
- DS8 pad 2: unconnected-(DS8-A-Pad2) -> Net-(DS8-A)
- DS9 pad 1: unconnected-(DS9-K-Pad1) -> B0out
- DS9 pad 2: unconnected-(DS9-A-Pad2) -> Net-(DS9-A)
- F1 pad 1: unconnected-(F1-Pad1) -> Net-(Q1-C)
- F1 pad 2: unconnected-(F1-Pad2) -> 24Vout
- J2 pad 1: unconnected-(J2-Pin_1-Pad1) -> GND
- J2 pad 10: unconnected-(J2-Pin_10-Pad10) -> B2out
- J2 pad 11: unconnected-(J2-Pin_11-Pad11) -> B1out
- J2 pad 12: unconnected-(J2-Pin_12-Pad12) -> B0out
- J2 pad 13: unconnected-(J2-Pin_13-Pad13) -> A7out
- J2 pad 14: unconnected-(J2-Pin_14-Pad14) -> A6out
- J2 pad 15: unconnected-(J2-Pin_15-Pad15) -> A5out
- J2 pad 16: unconnected-(J2-Pin_16-Pad16) -> A4out
- J2 pad 17: unconnected-(J2-Pin_17-Pad17) -> A3out
- J2 pad 18: unconnected-(J2-Pin_18-Pad18) -> A2out
- J2 pad 19: unconnected-(J2-Pin_19-Pad19) -> A1out
- J2 pad 2: unconnected-(J2-Pin_2-Pad2) -> AUD
- J2 pad 20: unconnected-(J2-Pin_20-Pad20) -> A0out
- J2 pad 21: unconnected-(J2-Pin_21-Pad21) -> 24Vout
- J2 pad 22: unconnected-(J2-Pin_22-Pad22) -> 24Vout
- J2 pad 23: unconnected-(J2-Pin_23-Pad23) -> 24Vout
- J2 pad 24: unconnected-(J2-Pin_24-Pad24) -> 24Vout
- J2 pad 25: unconnected-(J2-Pin_25-Pad25) -> 24R
- J2 pad 26: unconnected-(J2-Pin_26-Pad26) -> 24R
- J2 pad 3: unconnected-(J2-Pin_3-Pad3) -> GND
- J2 pad 4: unconnected-(J2-Pin_4-Pad4) -> GND
- J2 pad 7: unconnected-(J2-Pin_7-Pad7) -> B5out
- J2 pad 8: unconnected-(J2-Pin_8-Pad8) -> B4out
- J2 pad 9: unconnected-(J2-Pin_9-Pad9) -> B3out
- Q1 pad 1: unconnected-(Q1-B-Pad1) -> 24Vpu
- Q1 pad 2: unconnected-(Q1-C-Pad2) -> Net-(Q1-C)
- Q1 pad 3: unconnected-(Q1-E-Pad3) -> 24V
- R1 pad 1: unconnected-(R1-Pad1) -> 24Vpu
- R1 pad 2: unconnected-(R1-Pad2) -> Net-(C11-Pad1)
- R10 pad 1: unconnected-(R10-Pad1) -> Net-(U9--)
- R10 pad 2: unconnected-(R10-Pad2) -> Net-(C12-Pad1)
- R11 pad 1: unconnected-(R11-Pad1) -> 5V
- R11 pad 2: unconnected-(R11-Pad2) -> Net-(U6-Pin_14)
- R7 pad 1: unconnected-(R7-Pad1) -> AUD
- R8 pad 1: Net-(U9--) -> Net-(R8-Pad1)
- R9 pad 1: Net-(U9--) -> Net-(R8-Pad1)
- R9 pad 2: Net-(C12-Pad1) -> Net-(U9--)
- TP1 pad 1: unconnected-(TP1-Pad1) -> GND
- TP2 pad 1: unconnected-(TP2-Pad1) -> 5V
- TP3 pad 1: unconnected-(TP3-Pad1) -> 12V
- TP4 pad 1: unconnected-(TP4-Pad1) -> -12V
- TP5 pad 1: unconnected-(TP5-Pad1) -> 24Vout
- TP6 pad 1: unconnected-(TP6-Pad1) -> AUD
- U1 pad 1: unconnected-(U1-R1.1-Pad1) -> Net-(DS5-A)
- U1 pad 10: unconnected-(U1-R5.2-Pad10) -> 24Vout
- U1 pad 11: unconnected-(U1-R4.2-Pad11) -> 24Vout
- U1 pad 12: unconnected-(U1-R3.2-Pad12) -> 24Vout
- U1 pad 13: unconnected-(U1-R2.2-Pad13) -> 24Vout
- U1 pad 14: unconnected-(U1-R1.2-Pad14) -> 24Vout
- U1 pad 2: unconnected-(U1-R2.1-Pad2) -> Net-(DS6-A)
- U1 pad 3: unconnected-(U1-R3.1-Pad3) -> Net-(DS7-A)
- U1 pad 4: unconnected-(U1-R4.1-Pad4) -> Net-(DS4-A)
- U1 pad 5: unconnected-(U1-R5.1-Pad5) -> Net-(DS3-A)
- U1 pad 6: unconnected-(U1-R6.1-Pad6) -> Net-(DS2-A)
- U1 pad 7: unconnected-(U1-R7.1-Pad7) -> Net-(DS1-A)
- U1 pad 8: unconnected-(U1-R7.2-Pad8) -> 24Vout
- U1 pad 9: unconnected-(U1-R6.2-Pad9) -> 24Vout
- U11 pad 1: unconnected-(U11-I1-Pad1) -> PA6
- U11 pad 10: unconnected-(U11-O7-Pad10) -> A0out
- U11 pad 11: unconnected-(U11-O6-Pad11) -> A1out
- U11 pad 12: unconnected-(U11-O5-Pad12) -> A2out
- U11 pad 13: unconnected-(U11-O4-Pad13) -> A3out
- U11 pad 14: unconnected-(U11-O3-Pad14) -> A4out
- U11 pad 15: unconnected-(U11-O2-Pad15) -> A5out
- U11 pad 16: unconnected-(U11-O1-Pad16) -> A6out
- U11 pad 2: unconnected-(U11-I2-Pad2) -> PA5
- U11 pad 3: unconnected-(U11-I3-Pad3) -> PA4
- U11 pad 4: unconnected-(U11-I4-Pad4) -> PA3
- U11 pad 5: unconnected-(U11-I5-Pad5) -> PA2
- U11 pad 6: unconnected-(U11-I6-Pad6) -> PA1
- U11 pad 7: unconnected-(U11-I7-Pad7) -> PA0
- U11 pad 8: unconnected-(U11-GND-Pad8) -> 24R
- U11 pad 9: unconnected-(U11-COM-Pad9) -> 24Vout
- U12 pad 1: unconnected-(U12-I1-Pad1) -> PA7
- U12 pad 10: unconnected-(U12-O7-Pad10) -> B5out
- U12 pad 11: unconnected-(U12-O6-Pad11) -> B4out
- U12 pad 12: unconnected-(U12-O5-Pad12) -> B3out
- U12 pad 13: unconnected-(U12-O4-Pad13) -> B2out
- U12 pad 14: unconnected-(U12-O3-Pad14) -> B1out
- U12 pad 15: unconnected-(U12-O2-Pad15) -> B0out
- U12 pad 16: unconnected-(U12-O1-Pad16) -> A7out
- U12 pad 2: unconnected-(U12-I2-Pad2) -> PB0
- U12 pad 3: unconnected-(U12-I3-Pad3) -> PB1
- U12 pad 4: unconnected-(U12-I4-Pad4) -> PB2
- U12 pad 5: unconnected-(U12-I5-Pad5) -> PB3
- U12 pad 6: unconnected-(U12-I6-Pad6) -> PB4
- U12 pad 7: unconnected-(U12-I7-Pad7) -> PB5
- U12 pad 8: unconnected-(U12-GND-Pad8) -> 24R
- U12 pad 9: unconnected-(U12-COM-Pad9) -> 24Vout
- U13 pad 10: unconnected-(U13-Pad10) -> Net-(C11-Pad1)
- U13 pad 11: unconnected-(U13-Pad11) -> 5Vpu
- U13 pad 12: unconnected-(U13-Pad12) -> 5Vpu
- U13 pad 13: unconnected-(U13-Pad13) -> CA2
- U13 pad 14: unconnected-(U13G-VCC-Pad14) -> 5V
- U13 pad 7: unconnected-(U13G-GND-Pad7) -> GND
- U14 pad 1: unconnected-(U14-0-Pad1) -> Net-(U14-0)
- U14 pad 12: unconnected-(U14-A3-Pad12) -> CB2
- U14 pad 13: unconnected-(U14-A2-Pad13) -> GND
- U14 pad 14: unconnected-(U14-A1-Pad14) -> PB7
- U14 pad 15: unconnected-(U14-A0-Pad15) -> PB6
- U14 pad 16: unconnected-(U14-VCC-Pad16) -> 5V
- U14 pad 2: unconnected-(U14-1-Pad2) -> Net-(U14-1)
- U14 pad 3: unconnected-(U14-2-Pad3) -> Net-(U14-2)
- U14 pad 4: unconnected-(U14-3-Pad4) -> Net-(U14-3)
- U14 pad 8: unconnected-(U14-GND-Pad8) -> GND
- U16 pad 10: unconnected-(U16-Pad10) -> Net-(U14-2)
- U16 pad 15: unconnected-(U16-Pad15) -> Net-(U14-3)
- U16 pad 2: unconnected-(U16-Pad2) -> Net-(U14-0)
- U16 pad 7: unconnected-(U16-Pad7) -> Net-(U14-1)
- U2 pad 1: unconnected-(U2-R1.1-Pad1) -> 24Vout
- U2 pad 10: unconnected-(U2-R5.2-Pad10) -> Net-(DS12-A)
- U2 pad 11: unconnected-(U2-R4.2-Pad11) -> Net-(DS11-A)
- U2 pad 12: unconnected-(U2-R3.2-Pad12) -> Net-(DS10-A)
- U2 pad 13: unconnected-(U2-R2.2-Pad13) -> Net-(DS8-A)
- U2 pad 14: unconnected-(U2-R1.2-Pad14) -> Net-(DS9-A)
- U2 pad 2: unconnected-(U2-R2.1-Pad2) -> 24Vout
- U2 pad 3: unconnected-(U2-R3.1-Pad3) -> 24Vout
- U2 pad 4: unconnected-(U2-R4.1-Pad4) -> 24Vout
- U2 pad 5: unconnected-(U2-R5.1-Pad5) -> 24Vout
- U2 pad 6: unconnected-(U2-R6.1-Pad6) -> 24Vout
- U2 pad 7: unconnected-(U2-R7.1-Pad7) -> 24Vout
- U2 pad 8: unconnected-(U2-R7.2-Pad8) -> Net-(DS14-A)
- U2 pad 9: unconnected-(U2-R6.2-Pad9) -> Net-(DS13-A)
- U6 pad 1: unconnected-(U6-Pin_1-Pad1) -> BS1
- U6 pad 10: unconnected-(U6-Pin_10-Pad10) -> BS10
- U6 pad 14: unconnected-(U6-Pin_14-Pad14) -> Net-(U6-Pin_14)
- U6 pad 2: unconnected-(U6-Pin_2-Pad2) -> BS2
- U6 pad 3: unconnected-(U6-Pin_3-Pad3) -> BS3
- U6 pad 4: unconnected-(U6-Pin_4-Pad4) -> BS4
- U6 pad 5: unconnected-(U6-Pin_5-Pad5) -> BS5
- U6 pad 6: unconnected-(U6-Pin_6-Pad6) -> BS6
- U6 pad 7: unconnected-(U6-Pin_7-Pad7) -> BS7
- U6 pad 8: unconnected-(U6-Pin_8-Pad8) -> BS8
- U6 pad 9: unconnected-(U6-Pin_9-Pad9) -> BS9
- U7 pad 1: unconnected-(U7-VSS-Pad1) -> GND
- U7 pad 10: unconnected-(U7-PB0-Pad10) -> PB0
- U7 pad 11: unconnected-(U7-PB1-Pad11) -> PB1
- U7 pad 12: unconnected-(U7-PB2-Pad12) -> PB2
- U7 pad 13: unconnected-(U7-PB3-Pad13) -> PB3
- U7 pad 14: unconnected-(U7-PB4-Pad14) -> PB4
- U7 pad 15: unconnected-(U7-PB5-Pad15) -> PB5
- U7 pad 16: unconnected-(U7-PB6-Pad16) -> PB6
- U7 pad 17: unconnected-(U7-PB7-Pad17) -> PB7
- U7 pad 19: unconnected-(U7-CB2-Pad19) -> CB2
- U7 pad 2: unconnected-(U7-PA0-Pad2) -> PA0
- U7 pad 20: unconnected-(U7-VCC-Pad20) -> 5V
- U7 pad 21: unconnected-(U7-R/~{W}-Pad21) -> R/~{W}
- U7 pad 22: unconnected-(U7-CS0-Pad22) -> CS
- U7 pad 23: unconnected-(U7-~{CS2}-Pad23) -> Net-(U6-Pin_14)
- U7 pad 24: unconnected-(U7-CS1-Pad24) -> CS
- U7 pad 25: unconnected-(U7-ENABLE-Pad25) -> PHI2
- U7 pad 26: unconnected-(U7-D7-Pad26) -> DBB7
- U7 pad 27: unconnected-(U7-D6-Pad27) -> DBB6
- U7 pad 28: unconnected-(U7-D5-Pad28) -> DBB5
- U7 pad 29: unconnected-(U7-D4-Pad29) -> DBB4
- U7 pad 3: unconnected-(U7-PA1-Pad3) -> PA1
- U7 pad 30: unconnected-(U7-D3-Pad30) -> DBB3
- U7 pad 31: unconnected-(U7-D2-Pad31) -> DBB2
- U7 pad 32: unconnected-(U7-D1-Pad32) -> DBB1
- U7 pad 33: unconnected-(U7-D0-Pad33) -> DBB0
- U7 pad 34: unconnected-(U7-~{RESET}-Pad34) -> ~{MRST}
- U7 pad 35: unconnected-(U7-RS1-Pad35) -> BA1
- U7 pad 36: unconnected-(U7-RS0-Pad36) -> BA0
- U7 pad 39: unconnected-(U7-CA2-Pad39) -> CA2
- U7 pad 4: unconnected-(U7-PA2-Pad4) -> PA2
- U7 pad 5: unconnected-(U7-PA3-Pad5) -> PA3
- U7 pad 6: unconnected-(U7-PA4-Pad6) -> PA4
- U7 pad 7: unconnected-(U7-PA5-Pad7) -> PA5
- U7 pad 8: unconnected-(U7-PA6-Pad8) -> PA6
- U7 pad 9: unconnected-(U7-PA7-Pad9) -> PA7
- U8 pad 1: unconnected-(U8-R1.1-Pad1) -> CA2
- U8 pad 10: unconnected-(U8-R7.2-Pad10) -> 5V
- U8 pad 11: unconnected-(U8-R6.2-Pad11) -> 5V
- U8 pad 12: unconnected-(U8-R5.2-Pad12) -> 5V
- U8 pad 13: unconnected-(U8-R4.2-Pad13) -> 5V
- U8 pad 14: unconnected-(U8-R3.2-Pad14) -> 24V
- U8 pad 15: unconnected-(U8-R2.2-Pad15) -> 5V
- U8 pad 16: unconnected-(U8-R1.2-Pad16) -> 5V
- U8 pad 2: unconnected-(U8-R2.1-Pad2) -> 5Vpu
- U8 pad 3: unconnected-(U8-R3.1-Pad3) -> 24Vpu
- U8 pad 4: unconnected-(U8-R4.1-Pad4) -> CS
- U8 pad 5: unconnected-(U8-R5.1-Pad5) -> Net-(U14-3)
- U8 pad 6: unconnected-(U8-R6.1-Pad6) -> Net-(U14-2)
- U8 pad 7: unconnected-(U8-R7.1-Pad7) -> Net-(U14-1)
- U8 pad 8: unconnected-(U8-R8.1-Pad8) -> Net-(U14-0)
- U8 pad 9: unconnected-(U8-R8.2-Pad9) -> 5V
Routing:
- net AUD: track 0.00 -> 427.1 mm, vias 0 -> 2
- net 5V: track 0.00 -> 409.1 mm, vias 0 -> 4
- net 24Vout: track 0.00 -> 362.9 mm, vias 0 -> 6
- net GND: track 237.6 -> 578.6 mm, vias 4 -> 7
- net 12V: track 0.00 -> 304.6 mm, vias 0 -> 3
- net -12V: track 0.00 -> 282.1 mm, vias 0 -> 2
- net B5out: track 0.00 -> 216.5 mm
- net B4out: track 0.00 -> 215.2 mm
- net 24V: track 0.00 -> 208.0 mm, vias 0 -> 3
- net B3out: track 0.00 -> 207.4 mm
- net B2out: track 0.00 -> 205.8 mm
- net A7out: track 0.00 -> 202.1 mm, vias 0 -> 1
- net B0out: track 0.00 -> 199.6 mm
- net B1out: track 0.00 -> 197.6 mm
- net A6out: track 0.00 -> 192.1 mm
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- added copper zone on B.Cu, net GND
- added copper zone on F.Cu, net GND
- added copper zone on B.Cu, net Net-(Q1-C)
- added copper zone on F.Cu, net Net-(Q1-C)
Other:
- outline, holes or cut-outs redrawn
- board text added: "1"
- board text added: "25"
- board text added: "49"
- board text added: "ASSY 06-0004"
- board text added: "PART 07-0004 REV A"
- board text added: "PCB1-6"

Commit message: revised copper layer character card rev a
Other:
- board text added: "2"
- board text added: "50"
Changed lines of the file:
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@@
+    (effects (font (size 1.5 1.5) (thickness 0.3) bold) (justify left bottom mirror))
+  )
+  (gr_text "50" (at 182.245 93.98 90) (layer "B.Cu")
+    (effects (font (size 1.5 1.5) (thickness 0.3) bold) (justify left bottom mirror))
+  )
+  (gr_text "2" (at 182.88 10.16 90) (layer "B.Cu")
     (effects (font (size 1.5 1.5) (thickness 0.3) bold) (justify left bottom mirror))
   )
