File: Boards/Character board 0004 rev.a/Character board 0004 rev.a.kicad_sch (KiCad schematic)
At the start: 64 parts, among them J1 card edge, J2 character connector, Q1 2N6125, U1 2.2K, U1 6821, U13 7406, U14 74LS42, U15 LM741, U16 AH5012, U2 2.2K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

Commit message: updated boards to have correct logos
Parts:
- added TP2: GND, TestPoint:TestPoint_Plated_Hole_D3.0mm, symbol Connector:TestPoint
Connections:
- net A4out: now also DS1.1 (K); no longer DS1.1 (K)
- net A6out: now also DS1.1 (K); no longer DS1.1 (K)
- net GND: now also TP2.1
Changed lines of the file:
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@@
   (junction (at 229.235 159.385) (diameter 0) (color 0 0 0 0)
   )
+  (junction (at 219.075 92.71) (diameter 0) (color 0 0 0 0)
+  )
   (junction (at 219.075 218.44) (diameter 0) (color 0 0 0 0)
   )
@@
   (junction (at 213.995 118.11) (diameter 0) (color 0 0 0 0)
   )
+  (junction (at 252.095 242.57) (diameter 0) (color 0 0 0 0)
+  )
   (junction (at 182.245 113.03) (diameter 0) (color 0 0 0 0)
   )
@@
   (junction (at 83.185 64.135) (diameter 0) (color 0 0 0 0)
   )
-  (junction (at 229.235 92.71) (diameter 0) (color 0 0 0 0)
-  )
   (junction (at 213.995 151.765) (diameter 0) (color 0 0 0 0)
   )
@@
   (junction (at 66.675 19.05) (diameter 0) (color 0 0 0 0)
   )
-  (junction (at 219.075 97.79) (diameter 0) (color 0 0 0 0)
-  )
   (junction (at 182.88 69.85) (diameter 0) (color 0 0 0 0)
   )
@@
   (junction (at 285.75 188.595) (diameter 0) (color 0 0 0 0)
   )
+  (junction (at 229.235 97.79) (diameter 0) (color 0 0 0 0)
+  )
   (junction (at 194.945 19.05) (diameter 0) (color 0 0 0 0)
   )
@@
     (stroke (width 0) (type default))
   )
-  (wire (pts (xy 219.075 97.79) (xy 192.405 97.79))
-    (stroke (width 0) (type default))
-  )
   (wire (pts (xy 48.895 123.19) (xy 46.355 123.19))
     (stroke (width 0) (type default))
@@
     (stroke (width 0) (type default))
   )
-  (wire (pts (xy 235.585 92.71) (xy 229.235 92.71))
+  (wire (pts (xy 192.405 92.71) (xy 219.075 92.71))
     (stroke (width 0) (type default))
   )
@@
     (stroke (width 0) (type default))
   )
+  (wire (pts (xy 229.235 89.535) (xy 229.235 97.79))
+    (stroke (width 0) (type default))
+  )
   (wire (pts (xy 33.655 95.25) (xy 31.115 95.25))
     (stroke (width 0) (type default))
@@
     (stroke (width 0) (type default))
   )
-  (wire (pts (xy 229.235 92.71) (xy 229.235 89.535))
-    (stroke (width 0) (type default))
-  )
   (wire (pts (xy 221.615 128.27) (xy 229.235 128.27))
     (stroke (width 0) (type default))
@@
     (stroke (width 0) (type default))
   )
+  (wire (pts (xy 219.075 89.535) (xy 219.075 92.71))
+    (stroke (width 0) (type default))
+  )
+  (wire (pts (xy 219.075 92.71) (xy 235.585 92.71))
+    (stroke (width 0) (type default))
+  )
   (wire (pts (xy 71.12 55.88) (xy 83.185 55.88))
     (stroke (width 0) (type default))
@@
     (stroke (width 0) (type default))
   )
-  (wire (pts (xy 235.585 97.79) (xy 219.075 97.79))
+  (wire (pts (xy 192.405 97.79) (xy 229.235 97.79))
     (stroke (width 0) (type default))
   )
@@
     (stroke (width 0) (type default))
   )
-  (wire (pts (xy 229.235 92.71) (xy 192.405 92.71))
-    (stroke (width 0) (type default))
-  )
   (wire (pts (xy 253.365 172.72) (xy 253.365 177.8))
     (stroke (width 0) (type default))
@@
     (stroke (width 0) (type default))
   )
-  (wire (pts (xy 219.075 97.79) (xy 219.075 89.535))
-    (stroke (width 0) (type default))
-  )
   (wire (pts (xy 33.655 97.79) (xy 31.115 97.79))
     (stroke (width 0) (type default))
@@
     (stroke (width 0) (type default))
   )
+  (wire (pts (xy 229.235 97.79) (xy 235.585 97.79))
+    (stroke (width 0) (type default))
+  )
   (wire (pts (xy 33.655 130.81) (xy 31.115 130.81))
     (stroke (width 0) (type default))
@@
     (stroke (width 0) (type default))
   )
+  (wire (pts (xy 264.795 242.57) (xy 252.095 242.57))
+    (stroke (width 0) (type default))
+  )
   (wire (pts (xy 48.895 110.49) (xy 46.355 110.49))
     (stroke (width 0) (type default))
@@
         )
       )
+    )
+  )
+  (symbol (lib_id "Connector:TestPoint") (at 264.795 242.57 270) (mirror x) (unit 1)
+    (in_bom yes) (on_board yes) (dnp no) (fields_autoplaced)
+    (property "Reference" "TP2" (at 269.494 241.9263 90)
+      (effects (font (size 1.27 1.27)) (justify left))
+    )
+    (property "Value" "GND" (at 269.494 243.8473 90)
+      (effects (font (size 1.27 1.27)) (justify left))
+    )
+    (property "Footprint" "TestPoint:TestPoint_Plated_Hole_D3.0mm" (at 264.795 237.49 0)
+      (effects (font (size 1.27 1.27)) hide)
+    )
+    (property "Datasheet" "~" (at 264.795 237.49 0)
+      (effects (font (size 1.27 1.27)) hide)
+    )
+    (pin "1")
+    (instances
+      (project "Audio board rev.a"
+        (path "/439a8b7c-4c76-4152-9c42-79901501747e"
+          (reference "TP2") (unit 1)
+        )
+      )
+      (project "Character board 0004 rev.a"
+        (path "/cb28dba3-810b-45e4-988f-432ba6e2d266"
+          (reference "G1") (unit 1)
+        )
+      )
