File: Boards/Light board 0021 rev.0/Light board 0021 rev.0.kicad_pcb (KiCad board)
At the start: 2 copper layers, 166.4 x 186.7 mm, 65 parts, among them J1 card edge, J2 character connector, Q1 2N6125, U1 2.2K, U10 Unused DIP, U11 ULN2003A, U12 ULN2003A, U13 7406, U14 74LS42, U15 LM741, U16 AH5012, U2 2.2K, U3 Unused DIP, U4 Unused DIP, U5 Unused DIP, U6 Board ID header, U7 6821, U8 3.3K, U9 LM741

Commit message: almost done with the old light driver
Parts:
- removed C10: 10nF, Capacitor_THT:C_Rect_L7.0mm_W2.5mm_P5.00mm
- removed C12, C7, C8: 100nF, Capacitor_THT:C_Rect_L7.0mm_W2.5mm_P5.00mm
- removed the C3 at (176.5, 47.0)
- removed the C4 at (156.8, 47.0)
- removed C6: 1nF, Capacitor_THT:C_Rect_L9.0mm_W2.7mm_P7.50mm_MKT
- removed R10: 47.5K, Evan's parts:R_Axial_DIN0204_L3.6mm_D1.6mm_P12.7mm_Horizontal
- removed the R4 at (174.0, 20.3)
- removed R5, R6: 20.0K, Evan's parts:R_Axial_DIN0204_L3.6mm_D1.6mm_P12.7mm_Horizontal
- removed R7: 120, Evan's parts:R_Axial_DIN0204_L3.6mm_D1.6mm_P12.7mm_Horizontal
- removed R8: 100K, Potentiometer_THT:Potentiometer_Bourns_3005_Horizontal
- removed R9: 10.0K, Evan's parts:R_Axial_DIN0204_L3.6mm_D1.6mm_P12.7mm_Horizontal
- removed TP3: +12, TestPoint:TestPoint_Plated_Hole_D3.0mm
- removed TP4: -12, TestPoint:TestPoint_Plated_Hole_D3.0mm
- removed TP6: AUD, TestPoint:TestPoint_Plated_Hole_D3.0mm
- removed U10: Unused DIP, Package_DIP:DIP-16_W7.62mm
- removed U11, U12: ULN2003A, Package_DIP:DIP-16_W7.62mm
- removed U13: 7406, Package_DIP:DIP-14_W7.62mm
- removed U15, U9: LM741, Package_DIP:DIP-8_W7.62mm
- added DS15: LED, Evan's parts:LED_D5.0mm_Horizontal_O3.81mm_Z15.0mm reversed, F.Cu at (24.1, 45.7)
- added DS16: LED, Evan's parts:LED_D5.0mm_Horizontal_O3.81mm_Z15.0mm reversed, F.Cu at (24.1, 38.7)
- C3: renamed from C5; footprint Capacitor_THT:C_Rect_L7.0mm_W2.5mm_P5.00mm -> Capacitor_THT:C_Rect_L9.0mm_W2.5mm_P7.50mm_MKT
- C4: renamed from C11; footprint Capacitor_THT:C_Rect_L7.0mm_W2.5mm_P5.00mm -> Capacitor_THT:C_Rect_L9.0mm_W2.5mm_P7.50mm_MKT
- C5: renamed from C9; footprint Capacitor_THT:C_Rect_L7.0mm_W2.5mm_P5.00mm -> Capacitor_THT:C_Rect_L9.0mm_W2.5mm_P7.50mm_MKT
- J2: value character connector -> light connector; footprint Connector_PinHeader_2.54mm:PinHeader_2x13_P2.54mm_Horizontal -> Connector_PinHeader_2.54mm:PinHeader_2x25_P2.54mm_Horizontal
- R2, R3: value 20.0K -> 2.2K
- U14: value 74LS42 -> Unused DIP
- U16: value AH5012 -> Unused DIP
- U3, U4: value Unused DIP -> ULN2003A
- U5: value Unused DIP -> 7406; footprint Package_DIP:DIP-16_W7.62mm -> Package_DIP:DIP-14_W7.62mm
- moved R2 130.8 mm to (44.5, 45.7), turned to 0 degrees
- moved R3 130.4 mm to (44.5, 38.7), turned to 0 degrees
- moved C3 66.9 mm to (97.2, 162.6), turned to 90 degrees
- moved R1 61.4 mm to (71.1, 121.9)
- moved C4 60.4 mm to (97.2, 119.4), turned to -90 degrees
- moved J2 41.5 mm to (210.8, 102.9)
- moved C1 34.7 mm to (179.7, 83.2), turned to 90 degrees
- moved C2 33.4 mm to (167.0, 54.6)
- moved CR1 25.8 mm to (148.6, 108.6)
- moved R4 16.6 mm to (137.2, 94.6)
- moved F1 13.4 mm to (80.6, 131.4)
- moved C5 12.0 mm to (130.8, 62.2), turned to 90 degrees
- moved DS1 1.91 mm to (24.1, 143.5)
- moved DS10 1.91 mm to (24.1, 80.6)
- moved DS11 1.91 mm to (24.1, 73.7)
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- renumbered R11 to R4
Connections:
- C4 pad 1: Net-(C11-Pad1) -> Net-(C4-Pad1)
- J1 pad 2: BCLK -> aux1_AGC
- J1 pad 4: UNUSED1 -> aux2_AGC
- J2 pad 1: GND -> 24Vout
- J2 pad 10: B2out -> unconnected-(J2-Pin_10-Pad10)
- J2 pad 11: B1out -> unconnected-(J2-Pin_11-Pad11)
- J2 pad 12: B0out -> unconnected-(J2-Pin_12-Pad12)
- J2 pad 13: A7out -> unconnected-(J2-Pin_13-Pad13)
- J2 pad 14: A6out -> unconnected-(J2-Pin_14-Pad14)
- J2 pad 15: A5out -> unconnected-(J2-Pin_15-Pad15)
- J2 pad 16: A4out -> unconnected-(J2-Pin_16-Pad16)
- J2 pad 17: A3out -> B7out
- J2 pad 18: A2out -> unconnected-(J2-Pin_18-Pad18)
- J2 pad 19: A1out -> B6out
- J2 pad 2: AUD -> 24R
- J2 pad 20: A0out -> unconnected-(J2-Pin_20-Pad20)
- J2 pad 21: 24Vout -> B5out
- J2 pad 22: 24Vout -> unconnected-(J2-Pin_22-Pad22)
- J2 pad 23: 24Vout -> B4out
- J2 pad 24: 24Vout -> unconnected-(J2-Pin_24-Pad24)
- J2 pad 25: 24R -> B3out
- J2 pad 26: 24R -> unconnected-(J2-Pin_26-Pad26)
- J2 pad 3: GND -> unconnected-(J2-Pin_3-Pad3)
- J2 pad 4: GND -> 24R
- J2 pad 6: unconnected-(J2-Pin_6-Pad6) -> 24R
- J2 pad 7: B5out -> unconnected-(J2-Pin_7-Pad7)
- J2 pad 8: B4out -> 24R
- J2 pad 9: B3out -> unconnected-(J2-Pin_9-Pad9)
- R1 pad 2: Net-(C11-Pad1) -> Net-(C4-Pad1)
- R2 pad 1: BGOUT_AGC -> Net-(DS15-A)
- R2 pad 2: Net-(R2-Pad2) -> 24Vout
- R3 pad 1: R2R_audio_AGC -> Net-(DS16-A)
- R3 pad 2: Net-(R3-Pad2) -> 24Vout
- U14 pad 1: Net-(U14-0) -> unconnected-(U14-R1.1-Pad1)
- U14 pad 12: CB2 -> unconnected-(U14-R5.2-Pad12)
- U14 pad 13: GND -> unconnected-(U14-R4.2-Pad13)
- U14 pad 14: PB7 -> unconnected-(U14-R3.2-Pad14)
- U14 pad 15: PB6 -> unconnected-(U14-R2.2-Pad15)
- U14 pad 2: Net-(U14-1) -> unconnected-(U14-R2.1-Pad2)
- U14 pad 3: Net-(U14-2) -> unconnected-(U14-R3.1-Pad3)
- U14 pad 4: Net-(U14-3) -> unconnected-(U14-R4.1-Pad4)
- U16 pad 1: Net-(U15--) -> unconnected-(U16-R1.1-Pad1)
- U16 pad 10: Net-(U14-2) -> unconnected-(U16-R7.2-Pad10)
- U16 pad 11: Net-(R4-Pad2) -> unconnected-(U16-R6.2-Pad11)
- U16 pad 12: GND -> unconnected-(U16-R5.2-Pad12)
- U16 pad 13: GND -> unconnected-(U16-R4.2-Pad13)
- U16 pad 14: Net-(R5-Pad2) -> unconnected-(U16-R3.2-Pad14)
- U16 pad 15: Net-(U14-3) -> unconnected-(U16-R2.2-Pad15)
- U16 pad 16: Net-(U15--) -> unconnected-(U16-R1.2-Pad16)
- U16 pad 2: Net-(U14-0) -> unconnected-(U16-R2.1-Pad2)
- U16 pad 3: Net-(R2-Pad2) -> unconnected-(U16-R3.1-Pad3)
- U16 pad 4: GND -> unconnected-(U16-R4.1-Pad4)
- U16 pad 5: GND -> unconnected-(U16-R5.1-Pad5)
- U16 pad 6: Net-(R3-Pad2) -> unconnected-(U16-R6.1-Pad6)
- U16 pad 7: Net-(U14-1) -> unconnected-(U16-R7.1-Pad7)
- U16 pad 8: Net-(U15--) -> unconnected-(U16-R8.1-Pad8)
- U16 pad 9: Net-(U15--) -> unconnected-(U16-R8.2-Pad9)
- U3 pad 1: unconnected-(U3-R1.1-Pad1) -> PA0
- U3 pad 10: unconnected-(U3-R7.2-Pad10) -> A6out
- U3 pad 11: unconnected-(U3-R6.2-Pad11) -> A5out
- U3 pad 12: unconnected-(U3-R5.2-Pad12) -> A4out
- U3 pad 13: unconnected-(U3-R4.2-Pad13) -> A3out
- U3 pad 14: unconnected-(U3-R3.2-Pad14) -> A2out
- U3 pad 15: unconnected-(U3-R2.2-Pad15) -> A1out
- U3 pad 16: unconnected-(U3-R1.2-Pad16) -> A0out
- U3 pad 2: unconnected-(U3-R2.1-Pad2) -> PA1
- U3 pad 3: unconnected-(U3-R3.1-Pad3) -> PA2
- U3 pad 4: unconnected-(U3-R4.1-Pad4) -> PA3
- U3 pad 5: unconnected-(U3-R5.1-Pad5) -> PA4
- U3 pad 6: unconnected-(U3-R6.1-Pad6) -> PA5
- U3 pad 7: unconnected-(U3-R7.1-Pad7) -> PA6
- U3 pad 8: unconnected-(U3-R8.1-Pad8) -> 24R
- U3 pad 9: unconnected-(U3-R8.2-Pad9) -> 24Vout
- U4 pad 1: unconnected-(U4-R1.1-Pad1) -> PA7
- U4 pad 10: unconnected-(U4-R7.2-Pad10) -> B5out
- U4 pad 11: unconnected-(U4-R6.2-Pad11) -> B4out
- U4 pad 12: unconnected-(U4-R5.2-Pad12) -> B3out
- U4 pad 13: unconnected-(U4-R4.2-Pad13) -> B2out
- U4 pad 14: unconnected-(U4-R3.2-Pad14) -> B1out
- U4 pad 15: unconnected-(U4-R2.2-Pad15) -> B0out
- U4 pad 16: unconnected-(U4-R1.2-Pad16) -> A7out
- U4 pad 2: unconnected-(U4-R2.1-Pad2) -> PB0
- U4 pad 3: unconnected-(U4-R3.1-Pad3) -> PB1
- U4 pad 4: unconnected-(U4-R4.1-Pad4) -> PB2
- U4 pad 5: unconnected-(U4-R5.1-Pad5) -> PB3
- U4 pad 6: unconnected-(U4-R6.1-Pad6) -> PB4
- U4 pad 7: unconnected-(U4-R7.1-Pad7) -> PB5
- U4 pad 8: unconnected-(U4-R8.1-Pad8) -> 24R
- U4 pad 9: unconnected-(U4-R8.2-Pad9) -> 24Vout
- U5 pad 1: unconnected-(U5-R1.1-Pad1) -> PB7
- U5 pad 10: unconnected-(U5-R7.2-Pad10) -> Net-(C4-Pad1)
- U5 pad 11: unconnected-(U5-R6.2-Pad11) -> 5Vpu
- U5 pad 12: unconnected-(U5-R5.2-Pad12) -> 5Vpu
- U5 pad 13: unconnected-(U5-R4.2-Pad13) -> CA2
- U5 pad 14: unconnected-(U5-R3.2-Pad14) -> 5V
- U5 pad 2: unconnected-(U5-R2.1-Pad2) -> B7out
- U5 pad 3: unconnected-(U5-R3.1-Pad3) -> PB6
- U5 pad 4: unconnected-(U5-R4.1-Pad4) -> B6out
- U5 pad 7: unconnected-(U5-R7.1-Pad7) -> GND
- U8 pad 14: 24V -> 24Vpu
- U8 pad 3: 24Vpu -> 24V
- U8 pad 5: Net-(U14-3) -> unconnected-(U8-R5.1-Pad5)
- U8 pad 6: Net-(U14-2) -> unconnected-(U8-R6.1-Pad6)
- U8 pad 7: Net-(U14-1) -> unconnected-(U8-R7.1-Pad7)
- U8 pad 8: Net-(U14-0) -> unconnected-(U8-R8.1-Pad8)
Routing:
- net GND: track 578.5 -> 182.5 mm, vias 7 -> 1
- net AUD: track 388.9 -> 0.00 mm, vias 2 -> 0
- net 12V: track 296.0 -> 0.00 mm, vias 3 -> 0
- net -12V: track 266.2 -> 0.00 mm, vias 2 -> 0
- net B7out: track 0.00 -> 138.0 mm
- net B6out: track 0.00 -> 137.7 mm
- net Net-(R7-Pad2): track 100.6 -> 0.00 mm
- net Net-(R8-Pad1): track 94.6 -> 0.00 mm
- net Net-(U14-2): track 80.1 -> 0.00 mm
- net Net-(U14-3): track 78.2 -> 0.00 mm
- net A0out: track 162.7 -> 86.2 mm
- net Net-(Q1-C): track 120.2 -> 47.0 mm, vias 2 -> 0
- net A7out: track 181.9 -> 110.0 mm, vias 1 -> 0
- net Net-(U14-1): track 66.0 -> 0.00 mm, vias 2 -> 0
- net A2out: track 162.4 -> 97.1 mm
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- removed copper zone on B.Cu, net GND
Other:
- board text added: "ASSY 06-0021"
- board text added: "B"
- board text added: "E"
- board text removed: "25"
- board text removed: "ASSY 06-0004"
- board text removed: "PART 07-0004 REV B"
- board text removed: "SJC4A27-81 94V-0"
