File: Boards/Light board 0021 rev.0/Light board 0021 rev.0.kicad_sch (KiCad schematic)
At the start: 43 parts, among them J1 card edge, J2 character connector, Q1 2N6125, U1 2.2K, U1 6821, U13 7406, U2 2.2K, U4 ULN2003A, U6 Board ID header

Commit message: almost done with the old light driver
Parts:
- removed C25: 10nF, Capacitor_THT:C_Rect_L7.0mm_W2.5mm_P5.00mm, symbol Device:C
- removed J2: character connector, Connector_PinHeader_2.54mm:PinHeader_2x13_P2.54mm_Horizontal, symbol Connector_Generic:Conn_02x13_Odd_Even
- removed TP2: +12, TestPoint:TestPoint_Plated_Hole_D3.0mm, symbol Connector:TestPoint
- removed TP2: -12, TestPoint:TestPoint_Plated_Hole_D3.0mm, symbol Connector:TestPoint
- added DS1 (x2): LED, LED_THT:LED_D5.0mm_Horizontal_O3.81mm_Z15.0mm, symbol Device:LED
- added J2: light connector, Connector_PinHeader_2.54mm:PinHeader_2x25_P2.54mm_Horizontal, symbol Connector_Generic:Conn_02x25_Odd_Even
- added RP1: 3.3K, Package_DIP:DIP-16_W7.62mm, symbol Device:R_Pack08
- renumbered U13 to U5
Connections:
- net 24R: now also J2.2 (Pin_2), J2.4 (Pin_4), J2.6 (Pin_6), J2.8 (Pin_8)
- net 24V: now also RP1.3 (R3.1)
- net 24Vout: now also R33.2, R33.2, J2.1 (Pin_1), J2.49 (Pin_49)
- net 24Vpu: now also RP1.14 (R3.2)
- net 5V: now also RP1.16 (R1.2), RP1.10 (R7.2), RP1.11 (R6.2), RP1.12 (R5.2), RP1.13 (R4.2), RP1.15 (R2.2), RP1.16 (R1.2), RP1.9 (R8.2)
- net 5Vpu: now also RP1.2 (R2.1)
- net A0out: now also U4.16 (O1), J2.47 (Pin_47); no longer U4.10 (O7)
- net A1out: now also U4.15 (O2), J2.45 (Pin_45); no longer U4.11 (O6)
- net A2out: now also U4.14 (O3), J2.43 (Pin_43); no longer U4.12 (O5)
- net A3out: now also J2.41 (Pin_41)
- net A4out: now also DS1.1 (K), U4.12 (O5), J2.39 (Pin_39); no longer DS1.1 (K), U4.14 (O3)
- net A5out: now also U4.11 (O6), J2.37 (Pin_37); no longer U4.15 (O2)
- net A6out: now also DS1.1 (K), U4.10 (O7), J2.35 (Pin_35); no longer DS1.1 (K), U4.16 (O1)
- net A7out: now also J2.33 (Pin_33)
- net B0out: now also J2.31 (Pin_31)
- net B1out: now also J2.29 (Pin_29)
- net B2out: now also J2.27 (Pin_27)
- net B3out: now also J2.25 (Pin_25)
- net B4out: now also J2.23 (Pin_23)
- net B5out: now also J2.21 (Pin_21)
- net CA2: now also RP1.1 (R1.1)
- net CS: now also RP1.4 (R4.1)
- net GND: now also RP1.8 (R8.1)
- net PA0: now also U4.1 (I1); no longer U4.7 (I7)
- net PA1: now also U4.2 (I2); no longer U4.6 (I6)
- net PA2: now also U4.3 (I3); no longer U4.5 (I5)
- net PA4: now also U4.5 (I5); no longer U4.3 (I3)
- net PA5: now also U4.6 (I6); no longer U4.2 (I2)
- net PA6: now also U4.7 (I7); no longer U4.1 (I1)
- net PB6: now also U5.3
- net PB7: now also U5.1
- net B7out: now reaches U5.2
- net B7out: now also DS1.1 (K), J2.17 (Pin_17)
- net B6out: now reaches U5.4
- net B6out: now also DS1.1 (K), J2.19 (Pin_19)
- net at R33.1: now also DS1.2 (A) (x2)
- no-connect marks 49 -> 73
Other:
- moved on the sheet: R33, RP1, TP2, U5A, U5B, U5C, U5D
