File: Boards/Audio board 0003 rev.c/Audio board 0003 rev.c.kicad_sch (KiCad schematic)
At the start: 109 parts, among them J1 CEC card edge connector large, U1 6821, U10 LM324, U11 MC1458, U2 LM339, U3 LM339, U4 ULN2003A, U5 DAC-08, U6 DAC-08, U9 LM324

Commit message: finish light board rev.a, rename files, add renders and schematics, move pictures
Other:
- moved on the sheet: C1, C11, C12, C13, C14, C15, C16, C17, C18, C19, C2, C20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
