File: Boards/Audio board 0033 rev.a/Audio board 0033 rev.a.kicad_sch (KiCad schematic)
At the start: 104 parts, among them J1 CEC card edge connector large, U1 6821, U10 LM324, U11 MC1458, U2 LM339, U3 LM339, U4 ULN2003A, U5 DAC-08, U6 DAC-08, U7 AH5012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

Commit message: finish light board rev.a, rename files, add renders and schematics, move pictures
Connections:
- net CB2: now also C25.2, R25.2, R31.2, U7.11, U7.16, U7.9, U9.6 (-)
Other:
- moved on the sheet: C1, C11, C12, C13, C14, C15, C16, C17, C18, C19, C2, C20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
