File: Boards/Transpoart board 0020 rev.1982/Transpoart board 0020 rev.1982.kicad_sch (KiCad schematic)
At the start: 41 parts, among them J1 CEC card edge connector large, U1 6821, U10 LM311, U11 LM741, U12 LM311, U4 ULN2003A, U5 74LS74, U7 AH5012

Commit message: finished schematic (incorrect) digitization
Parts:
- added C21: 4.7uF, Evan's parts:CP_Radial_Tantal_D4mm_P3.81mm, symbol Device:C_Polarized
- added C34 (x5): 100nF, Capacitor_THT:C_Rect_L9.0mm_W2.5mm_P7.50mm_MKT, symbol Device:C
- added C34: 50nF, Capacitor_THT:C_Rect_L9.0mm_W2.5mm_P7.50mm_MKT, symbol Device:C
- added C34: 20nF, Capacitor_THT:C_Rect_L9.0mm_W2.5mm_P7.50mm_MKT, symbol Device:C
- added C4 (x2): 100nF, Capacitor_THT:C_Disc_D3.0mm_W1.6mm_P2.50mm, symbol Device:C
- added C7 (x3): 100pF, Capacitor_THT:C_Rect_L7.0mm_W2.5mm_P5.00mm, symbol Device:C
- added C7: 3300pF, Capacitor_THT:C_Rect_L7.0mm_W2.5mm_P5.00mm, symbol Device:C
- added R37 (x5): 10K, Resistor_THT:R_Axial_DIN0309_L9.0mm_D3.2mm_P12.70mm_Horizontal, symbol Device:R
- added R37: 2.2K, Resistor_THT:R_Axial_DIN0309_L9.0mm_D3.2mm_P12.70mm_Horizontal, symbol Device:R
- added R37: 470, Resistor_THT:R_Axial_DIN0309_L9.0mm_D3.2mm_P12.70mm_Horizontal, symbol Device:R
- added R37 (x2): 470K, Resistor_THT:R_Axial_DIN0309_L9.0mm_D3.2mm_P12.70mm_Horizontal, symbol Device:R
- added R37 (x3): 1K, Resistor_THT:R_Axial_DIN0309_L9.0mm_D3.2mm_P12.70mm_Horizontal, symbol Device:R
- added R37: 100K, Resistor_THT:R_Axial_DIN0309_L9.0mm_D3.2mm_P12.70mm_Horizontal, symbol Device:R
- added R37 (x2): 4.7K, Resistor_THT:R_Axial_DIN0309_L9.0mm_D3.2mm_P12.70mm_Horizontal, symbol Device:R
- added R37: 39K, Resistor_THT:R_Axial_DIN0309_L9.0mm_D3.2mm_P12.70mm_Horizontal, symbol Device:R
- added R38: 5K, Potentiometer_THT:Potentiometer_Bourns_3005_Horizontal, symbol Device:R_Potentiometer
- added TP7: ones?, TestPoint:TestPoint_Plated_Hole_D3.0mm, symbol Connector:TestPoint
- added TP7: pulses, TestPoint:TestPoint_Plated_Hole_D3.0mm, symbol Connector:TestPoint
- added TP7: zeroes?, TestPoint:TestPoint_Plated_Hole_D3.0mm, symbol Connector:TestPoint
- added TP7: second filtered audio, TestPoint:TestPoint_Plated_Hole_D3.0mm, symbol Connector:TestPoint
- added TP7: filtered audio, TestPoint:TestPoint_Plated_Hole_D3.0mm, symbol Connector:TestPoint
- added U1: TR1602, Package_DIP:DIP-40_W15.24mm, symbol Evan's parts:TR1602
- added U3, U7: DM8602N, symbol Evan's parts:DM8602N
- added U4: 7410, symbol 74xx:74LS10
- added unit 2 of U4
- added unit 4 of U4
- added unit 3 of U4
- added unit 2 of U7
- added unit 3 of U7
- added U8: 74LS00, symbol 74xx:74LS00
Connections:
- net +12V: now also U10.8 (V+), U11.7 (V+), U12.8 (V+), C34.1, C4.2, C4.2, R37.1, R37.2
- net +5V: now also U5.14 (VCC), R37.1, R37.1, R37.1, R37.1, R37.2, R38.3, U1.1 (VSS), U3.16 (VCC), U4.14 (VCC), U7.16 (VCC), U8.14 (VCC)
- net -12V: now also U10.4 (V-), U11.4 (V-), U12.4 (V-), C34.1, U1.2 (VGG)
- net AUDIO IN: now also C34.1
- net BCLK: now also U1.17 (RCK), U1.40 (TCK)
- net CA2: now also U1.18 (~{DDR})
- net CB2: now also U1.23 (~{THRL})
- net DATA OUT: now also U8.11
- net GND: now also U10.1 (GND), U12.1 (GND), U5.2 (D), U5.7 (GND), C21.2, C34.2, C34.2, C34.2, C34.2, C7.1, C7.1, R37.2, R37.2, R37.2, U1.16 (SFD), U1.3 (VDD), U1.39 (SFE), U3.12 (B), U3.8 (GND), U4.7 (GND), U7.4 (B), U7.8 (GND), U8.7 (GND)
- net PA0: now also U1.12 (R0), U1.26 (T0)
- net PA1: now also U1.11 (R1), U1.27 (T1)
- net PA2: now also U1.10 (R2), U1.28 (T2)
- net PA3: now also U1.29 (T3), U1.9 (R3)
- net PA4: now also U1.30 (T4), U1.8 (R4)
- net PA5: now also U1.31 (T5), U1.7 (R5)
- net PA6: now also U1.32 (T6), U1.6 (R6)
- net PA7: now also U1.33 (T7), U1.5 (R7)
- net PB0: now also U4.6 (I6), TP7.1, U3.10 (Q)
- net PB1: now also U1.24 (TRE)
- net PB2: now also U1.21 (MR)
- net PB3: now also U1.4 (~{RCVEN}), U8.1, U8.10, U8.2
- net PB4: now also U4.2 (I2)
- net PB5: now also U4.3 (I3)
- net PB6: now also U4.4 (I4)
- net PB7: now also U4.5 (I5)
- net pup: now also U5.1 (~{R}), U5.10 (~{S}), U5.13 (~{R}), R37.2, U1.34 (CRL), U1.35 (PI), U1.36 (SBS), U1.37 (WS1), U1.38 (WS2), U3.13 (Clr), U7.13 (Clr), U7.3 (Clr)
- net U9in: now reaches U4.1 (I1)
- net U9in: now also U5.3 (C), U4.6
- net U9out: now reaches U4.16 (O1)
- net U9out: now also U5.11 (C), R37.1
- net at U4.7 (I7): now also U5.8 (~{Q}), U8.5
- net at U10.2 (+): now also U12.3 (-), C7.2, R37.2, TP7.1
- net at U10.3 (-): now also C34.1, R37.1, R37.2
- net at U10.6 (STRB): now also C4.1
- net at U10.7: now also U12.7, R37.2, U7.5 (A)
- net at U11.2 (-): now also C7.1, R37.1, R37.2
- net at U11.3 (+): now also C7.2, R37.1, R37.1, R37.2
- net at U11.6: now also C7.2, R37.1, R37.1, TP7.1
- net at U5.12 (D): now also U5.5 (Q)
- net at U5.4 (~{S}): now also U4.12
- net at U7.14, U7.3: now also R37.2
- net CB1: now reaches U1.18 (CB1)
- net CB1: now also TP7.1, U4.2, U7.10 (Q), U7.12 (B)
- net CA1: now reaches U1.40 (CA1)
- net CA1: now also U1.19 (~{DR})
- net at U12.2 (+): now also C34.1, R37.1, R37.1
- net at U12.6 (STRB): now also C4.1
- new net: TP7.1, U3.11 (A), U4.1, U4.13, U4.3, U4.4, U4.5, U7.11 (A), U7.6 (Q), U7.9 (~{Q})
- new net: C34.1, R37.2, U3.14 (RCext)
- new net: C34.2, U3.15 (Cext)
- new net: C7.2, R37.2, U7.2 (RCext)
- new net: U8.3, U8.4
- new net: U8.12, U8.8
- new net: U1.25 (TO), U8.9
- new net: R37.1, R38.1, R38.2
- new net: C34.2, R37.1
- new net: U8.13, U8.6
- new net: C34.1, R37.2, U7.14 (RCext)
- new net: C34.2, U7.15 (Cext)
- new net: C7.1, U7.1 (Cext)
- no-connect marks 74 -> 94
Other:
- note added: "9600 Baud"
- moved on the sheet: C21, C34, C4, DS2, DS3, DS4, DS5, DS6, DS7, J1, RP1, TP2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
