File: Boards/Transpoart board 0020 rev.b/Transpoart board 0020 rev.b.kicad_sch (KiCad schematic)
At the start: 80 parts, among them J1 CEC card edge connector large, U1 6821, U1 TR1602, U10 LM311, U11 LM741, U12 LM311, U3 DM8602N, U4 7410, U4 ULN2003A, U5 74LS74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

Commit message: transport card digital section almost done
Parts:
- added C34: 10nF, Capacitor_THT:C_Rect_L7.2mm_W2.5mm_P5.00mm_FKS2_FKP2_MKS2_MKP2, symbol Device:C
- added U6: 74161, Package_DIP:DIP-16_W7.62mm, symbol 74xx:74LS161
- C34: footprint Capacitor_THT:C_Rect_L9.0mm_W2.5mm_P7.50mm_MKT -> Capacitor_THT:C_Rect_L7.2mm_W2.5mm_P5.00mm_FKS2_FKP2_MKS2_MKP2
- C34: value 20nF -> 39nF; footprint Capacitor_THT:C_Rect_L9.0mm_W2.5mm_P7.50mm_MKT -> Capacitor_THT:CP_Axial_L11.0mm_D6.0mm_P18.00mm_Horizontal
Connections:
- net +5V: now also C34.1, U6.16 (VCC)
- net BCLK: now also U4.9, U6.11 (Q3); no longer J1.62 (Pin_62)
- net DATA OUT: now also U1.25 (TO)
- net GND: now also C34.2, U6.3 (D0), U6.5 (D2), U6.6 (D3), U6.8 (GND)
- net PHI2: now also U6.2 (CP)
- net pup: now also U6.10 (CET)
- net at U4.7 (I7), U5.8 (~{Q}): now also U1.20 (RI)
- net at U4.10: now also U6.12 (Q2)
- net at U4.11: now also U6.13 (Q1)
- net at U4.8: now also U6.9 (~{PE})
- new net: U6.1 (~{MR}), U6.4 (D1), U6.7 (CEP)
- no-connect marks 128 -> 125
Other:
- note added: "?"
- note added: "guess"
- note added: "wrong ref des"
- note removed: "9600 Baud"
- moved on the sheet: U4C
