File: Boards/Transpoart board 0020 rev.b/Transpoart board 0020 rev.b.kicad_pcb (KiCad board)
At the start: 2 copper layers, 165.9 x 187.4 mm, 82 parts, among them P1 CEC card edge connector large, U1 TR1602, U10 LM311, U11 LM741, U12 LM311, U14 Spare, U15 Spare, U2 6821, U3 DM8602N, U4 7410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

Commit message: revised test point names
Parts:
- TP6: value pulses -> zero crossings
- TP7: value ones? -> bits
- TP8: value zeroes? -> carrier detect
Changed lines of the file:
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@@
         (effects (font (size 1 1) (thickness 0.15)))
     )
-    (fp_text value "pulses" (at 5.08 0) (layer "F.SilkS") hide
+    (fp_text value "zero crossings" (at 5.08 0) (layer "F.SilkS") hide
         (effects (font (size 1 1) (thickness 0.15)))
     )
@@
         (effects (font (size 1 1) (thickness 0.15)))
     )
-    (fp_text value "zeroes?" (at 5.08 0) (layer "F.SilkS") hide
+    (fp_text value "carrier detect" (at 5.08 0) (layer "F.SilkS") hide
         (effects (font (size 1 1) (thickness 0.15)))
     )
@@
         (effects (font (size 1 1) (thickness 0.15)))
     )
-    (fp_text value "ones?" (at 5.08 0) (layer "F.SilkS") hide
+    (fp_text value "bits" (at 5.08 0) (layer "F.SilkS") hide
         (effects (font (size 1 1) (thickness 0.15)))
     )
