File: Boards/Transpoart board 0020 rev.d/Transpoart board 0020 rev.d.kicad_pcb (KiCad board)
At the start: 2 copper layers, 165.9 x 187.4 mm, 82 parts, among them P1 CEC card edge connector large, U1 TR1602, U10 LM311, U11 LM741, U12 LM311, U14 Spare, U15 Spare, U2 6821, U3 DM8602N, U4 7410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

Commit message: rev.b and rev.d transport cards done?
Parts:
- added R17: 2.2K, Evan's parts:R_Axial_DIN0204_L3.6mm_D1.6mm_P12.7mm_Horizontal, F.Cu at (162.6, 167.6)
- added U13: AH5012, Package_DIP:DIP-16_W7.62mm, F.Cu at (118.7, 138.4)
Routing:
- net Net-(R17-Pad2): track 0.00 -> 63.7 mm
- net R.W.: track 219.6 -> 254.4 mm, vias 1 -> 3
- net F.F.: track 222.6 -> 243.7 mm, vias 1 -> 2
- net Net-(U11-+): track 14.6 -> 30.2 mm
- net GND: track 903.6 -> 911.2 mm
- net PLAY: track 220.6 -> 223.2 mm
- net STOP: track 228.4 -> 229.5 mm
Other:
- board text added: "ASSY 06-0020 REV D"
- board text added: "PN 007-0020 REV D"
- board text added: "SBC-A2 06-82"
- board text added: "TRANSPORT CONTROL"
- board text removed: "02-82"
- board text removed: "PART 07-0020 REV B"
- board text removed: "REV B ASSY 06-0020"
- board text removed: "SJC-4A/94V-0"

Commit message: revised test point names
Parts:
- TP6: value pulses -> zero crossings
- TP7: value ones? -> bits
- TP8: value zeroes? -> carrier detect
Changed lines of the file:
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@@
         (effects (font (size 1 1) (thickness 0.15)))
     )
-    (fp_text value "pulses" (at 5.08 0) (layer "F.SilkS") hide
+    (fp_text value "zero crossings" (at 5.08 0) (layer "F.SilkS") hide
         (effects (font (size 1 1) (thickness 0.15)))
     )
@@
         (effects (font (size 1 1) (thickness 0.15)))
     )
-    (fp_text value "zeroes?" (at 5.08 0) (layer "F.SilkS") hide
+    (fp_text value "carrier detect" (at 5.08 0) (layer "F.SilkS") hide
         (effects (font (size 1 1) (thickness 0.15)))
     )
@@
         (effects (font (size 1 1) (thickness 0.15)))
     )
-    (fp_text value "ones?" (at 5.08 0) (layer "F.SilkS") hide
+    (fp_text value "bits" (at 5.08 0) (layer "F.SilkS") hide
         (effects (font (size 1 1) (thickness 0.15)))
     )
