File: Boards/Transpoart board 0020 rev.d/Transpoart board 0020 rev.d.kicad_sch (KiCad schematic)
At the start: 81 parts, among them J1 CEC card edge connector large, U1 6821, U1 TR1602, U10 LM311, U11 LM741, U12 LM311, U3 DM8602N, U4 7410, U4 ULN2003A, U5 74LS74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

Commit message: rev.b and rev.d transport cards done?
Parts:
- added R37: 2.2K, Resistor_THT:R_Axial_DIN0309_L9.0mm_D3.2mm_P12.70mm_Horizontal, symbol Device:R
- added U7: AH5012, Package_DIP:DIP-16_W7.62mm, symbol Evan's parts:AH5012
Connections:
- net F.F.: now also U7.15
- net GND: now also U7.1, U7.16
- net R.W.: now also U7.2
- net at C7.2, R37.1, R37.2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: now also R37.1
- new net: R37.2, U7.14, U7.3
Other:
- moved on the sheet: U4C, U6

Commit message: revised test point names
Parts:
- TP7: value ones? -> bits
- TP7: value pulses -> zero crossings
- TP7: value zeroes? -> carrier detect
Changed lines of the file:
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@@
       (effects (font (size 1.27 1.27)) (justify left))
     )
-    (property "Value" "ones?" (at 221.742 60.2053 0)
+    (property "Value" "bits" (at 221.742 60.2053 0)
       (effects (font (size 1.27 1.27)) (justify left))
     )
@@
       (effects (font (size 1.27 1.27)) (justify left))
     )
-    (property "Value" "pulses" (at 250.952 58.9353 0)
+    (property "Value" "zero crossings" (at 250.952 58.9353 0)
       (effects (font (size 1.27 1.27)) (justify left))
     )
@@
       (effects (font (size 1.27 1.27)) (justify left))
     )
-    (property "Value" "zeroes?" (at 215.392 125.6103 0)
-      (effects (font (size 1.27 1.27)) (justify left))
-    )
+    (property "Value" "carrier detect" (at 215.392 125.6103 0)
+      (effects (font (size 1.27 1.27)) (justify left))
+    )
