File: Boards/CPU board 0001 rev.a/CPU board 0001 rev.a.kicad_sch (KiCad schematic)
At the start: 21 parts, among them J1 CEC card edge connector large, U1 LM7905_TO220

Commit message: half done routing cpu rev.a
Parts:
- added C2: 10pF, Capacitor_THT:C_Rect_L7.2mm_W2.5mm_P5.00mm_FKS2_FKP2_MKS2_MKP2, symbol Device:C
- added C21: 220uF, Capacitor_THT:CP_Axial_L29.0mm_D10.0mm_P35.00mm_Horizontal, symbol Device:C_Polarized
- added CR1, CR2, CR3, CR4, CR5, CR6: 1N914, Diode_THT:D_DO-35_SOD27_P7.62mm_Horizontal, symbol Diode:1N914
- added DS2 (x2), DS3 (x2), DS4, DS5, DS6, DS7: LED, LED_THT:LED_D5.0mm_Horizontal_O3.81mm_Z15.0mm, symbol Device:LED
- added R37 (x7): 4.7K, Resistor_THT:R_Axial_DIN0309_L9.0mm_D3.2mm_P12.70mm_Horizontal, symbol Device:R
- added R37: 330K, Resistor_THT:R_Axial_DIN0309_L9.0mm_D3.2mm_P12.70mm_Horizontal, symbol Device:R
- added R37: 100, Resistor_THT:R_Axial_DIN0309_L9.0mm_D3.2mm_P12.70mm_Horizontal, symbol Device:R
- added RP1, RP2: 10K, Package_DIP:DIP-16_W7.62mm, symbol Device:R_Pack08
- added RP1 (x4): SPARE, Package_DIP:DIP-16_W7.62mm, symbol Device:R_Pack08
- added TP2: IRQ, TestPoint:TestPoint_Plated_Hole_D3.0mm, symbol Connector:TestPoint
- added TP2: U18 CS, TestPoint:TestPoint_Plated_Hole_D3.0mm, symbol Connector:TestPoint
- added TP2: U19 CS, TestPoint:TestPoint_Plated_Hole_D3.0mm, symbol Connector:TestPoint
- added U10: 7432, Package_DIP:DIP-14_W7.62mm, symbol 74xx:74LS32
- added U11, U14, U15: 7442, Package_DIP:DIP-16_W7.62mm, symbol 74xx:74LS42
- added U12, U13, U8: 7406, Package_DIP:DIP-14_W7.62mm, symbol 74xx:74LS06
- added U16, U17: M8216, Package_DIP:DIP-16_W7.62mm, symbol Evan's parts:M8216
- added U18, U19: 6532, Package_DIP:DIP-40_W15.24mm, symbol cbm:6532
- added U20, U21, U22: 2708, Package_DIP:DIP-24_W15.24mm, symbol Evan's parts:2708
- added U23, U24, U5: 74367, Package_DIP:DIP-16_W7.62mm, symbol 74xx:74LS367
- added U25: 6502, Package_DIP:DIP-40_W15.24mm, symbol cbm:6502
- added U6: 7414, Package_DIP:DIP-14_W7.62mm, symbol 74xx:74LS14
- added U9: 7408, Package_DIP:DIP-14_W7.62mm, symbol 74xx:74LS08
- added W1: IRQ, Connector_PinSocket_2.54mm:PinSocket_2x01_P2.54mm_Vertical, symbol Connector_Generic:Conn_02x01
- added XU1: IC Socket, Package_DIP:DIP-16_W7.62mm, symbol Device:R_Pack08
- added Y1: 1Mhz, Crystal:Crystal_HC33-U_Horizontal, symbol Device:Crystal
- TP2: value GND -> ~{0/2/4}
- U7: renamed from U1; footprint Package_TO_SOT_THT:TO-220-3_Vertical -> Package_TO_SOT_THT:TO-220-3_Horizontal_TabDown
Connections:
- net +12V: now also U20.19 (VDD), U21.19 (VDD), U22.19 (VDD)
- net +5V: now also CR2.1 (K), CR3.1 (K), R37.1, R37.1, R37.1, R37.1, R37.1, R37.1, R37.1, RP1.1 (R1.1), RP1.16 (R1.2), RP1.16 (R1.2), RP1.16 (R1.2), RP1.16 (R1.2), RP1.2 (R2.1), RP1.3 (R3.1), RP1.4 (R4.1), RP1.5 (R5.1), RP1.6 (R6.1), RP1.7 (R7.1), RP1.8 (R8.1), RP2.10 (R7.2), RP2.11 (R6.2), RP2.12 (R5.2), RP2.13 (R4.2), RP2.14 (R3.2), RP2.15 (R2.2), RP2.16 (R1.2), RP2.9 (R8.2), U10.14 (VCC), U11.16 (VCC), U12.14 (VCC), U13.14 (VCC), U14.16 (VCC), U15.16 (VCC), U16.16 (VCC), U17.16 (VCC), U18.20 (Vcc), U19.20 (Vcc), U20.24 (VCC), U21.24 (VCC), U22.24 (VCC), U23.16 (VCC), U24.16 (VCC), U25.8 (Vcc), U5.16 (VCC), U6.14 (VCC), U8.14 (VCC), U9.14 (VCC)
- net -5V: now also U20.21 (VBB), U21.21 (VBB), U22.21 (VBB)
- net A0: now also U24.12 (I5), U25.9 (A0); no longer J1.75 (Pin_75)
- net A1: now also U24.4 (I2), U25.10 (A1); no longer J1.15 (Pin_15)
- net A10: now also U24.6 (I3), U25.19 (A10); no longer J1.30 (Pin_30)
- net A11: now also U24.10 (I4), U25.20 (A11); no longer J1.91 (Pin_91)
- net A12: now also U25.22 (A12), U5.12 (I5); no longer J1.31 (Pin_31)
- net A2: now also U24.14 (I6), U25.11 (A2); no longer J1.76 (Pin_76)
- net A3: now also U24.2 (I1), U25.12 (A3); no longer J1.16 (Pin_16)
- net A4: now also U23.10 (I4), U25.13 (A4); no longer J1.27 (Pin_27)
- net A5: now also U23.6 (I3), U25.14 (A5); no longer J1.88 (Pin_88)
- net A6: now also U23.4 (I2), U25.15 (A6); no longer J1.28 (Pin_28)
- net A7: now also U23.2 (I1), U25.16 (A7); no longer J1.89 (Pin_89)
- net A8: now also U23.14 (I6), U25.17 (A8); no longer J1.29
- net A9: now also U23.12 (I5), U25.18 (A9); no longer J1.90 (Pin_90)
- net AUDIO: now also U15.9 (7)
- net BS1: now also U11.1 (0)
- net BS10: now also U11.11 (9)
- net BS2: now also U11.2 (1)
- net BS3: now also U11.3 (2)
- net BS4: now also U11.4 (3)
- net BS5: now also U11.5 (4)
- net BS6: now also U11.6 (5)
- net BS7: now also U11.7 (6)
- net BS8: now also U11.9 (7)
- net BS9: now also U11.10 (8)
- net D0: now also U17.11 (DO2), U17.9 (DI2), U18.33 (D0), U19.33 (D0), U20.9 (D0), U21.9 (D0), U22.9 (D0), XU1.16 (R1.2); no longer J1.10 (Pin_10)
- net D1: now also U17.12 (DI3), U17.14 (DO3), U18.32 (D1), U19.32 (D1), U20.10 (D1), U21.10 (D1), U22.10 (D1), XU1.15 (R2.2); no longer J1.71 (Pin_71)
- net D2: now also U17.2 (DO0), U17.4 (DI0), U18.31 (D2), U19.31 (D2), U20.11 (D2), U21.11 (D2), U22.11 (D2), XU1.14 (R3.2); no longer J1.11 (Pin_11)
- net D3: now also U17.5 (DO1), U17.7 (DI1), U18.30 (D3), U19.30 (D3), U20.13 (D3), U21.13 (D3), U22.13 (D3), XU1.13 (R4.2); no longer J1.72 (Pin_72)
- net D4: now also U16.11 (DO2), U16.9 (DI2), U18.29 (D4), U19.29 (D4), U20.14 (D4), U21.14 (D4), U22.14 (D4), XU1.12 (R5.2); no longer J1.12 (Pin_12)
- net D5: now also U16.12 (DI3), U16.14 (DO3), U18.28 (D5), U19.28 (D5), U20.15 (D5), U21.15 (D5), U22.15 (D5), XU1.11 (R6.2); no longer J1.73 (Pin_73)
- net D6: now also U16.2 (DO0), U16.4 (DI0), U18.27 (D6), U19.27 (D6), U20.16 (D6), U21.16 (D6), U22.16 (D6), XU1.10 (R7.2); no longer J1.13 (Pin_13)
- net D7: now also U16.5 (DO1), U16.7 (DI1), U18.26 (D7), U19.26 (D7), U20.17 (D7), U21.17 (D7), U22.17 (D7), XU1.9 (R8.2); no longer J1.74 (Pin_74)
- net GND: now also C34.2, C21.2, CR1.2 (A), RP1.8 (R8.1), RP1.8 (R8.1), RP1.8 (R8.1), RP1.8 (R8.1), U10.7 (GND), U11.8 (GND), U12.7 (GND), U13.7 (GND), U14.12 (A3), U14.8 (GND), U15.8 (GND), U16.8 (GND), U17.8 (GND), U18.1 (GND), U19.1 (GND), U20.12 (GND), U20.18 (PGM), U21.12 (GND), U21.18 (PGM), U22.12 (GND), U22.18 (PGM), U23.8 (GND), U24.8 (GND), U25.1 (VSS), U25.21 (GND), U5.8 (GND), U6.7 (GND), U8.7 (GND), U9.7 (GND)
- net PHI2: now also U18.39 (CA2), U19.39 (CA2), U6.8
- net RDY: now also R37.2, U25.2 (RDY)
- net R/~{W}: now also U18.35 (R/~{W}), U19.35 (R/~{W}), U5.13 (O6b), U9.10
- net UART: now also U15.3 (2)
- net XPRT: now also U15.7 (6)
- net /IRQ: now also R37.2, TP2.1, U18.25 (~{IRQ}), U19.25 (~{IRQ}), U25.4 (~{IRQ}), W1.1 (Pin_1); no longer J1.36 (Pin_36)
- net /RESET: now also R37.1, U18.34 (~{RESET}), U19.34 (~{RESET}), U25.40 (~{RESET}), U6.6
- net at TP2.1: now also CR4.1 (K), CR5.1 (K), CR6.1 (K)
- net PROG in: now reaches C34.1
- net PROG in: now also J1.48 (Pin_48), U18.15 (PA7)
- net NEXT out: now reaches J1.113 (Pin_113)
- net NEXT out: now also U12.4
- net PROG out: now reaches J1.114 (Pin_114)
- net PROG out: now also U13.6
- net AGC 4: now reaches J1.115 (Pin_115)
- net AGC 4: now also U19.14 (PA6)
- net AGC 1: now reaches J1.116 (Pin_116)
- net AGC 1: now also U19.12 (PA4)
- net INTRO out: now reaches J1.117 (Pin_117)
- net INTRO out: now also U12.10
- net SPEC out: now reaches J1.121 (Pin_121)
- net SPEC out: now also U12.8
- net DIAG out: now reaches J1.37 (Pin_37)
- net DIAG out: now also U12.6
- net MIKE SW.: now reaches J1.42 (Pin_42)
- net MIKE SW.: now also U19.8 (PA0)
- net CHEER in: now reaches J1.43 (Pin_43)
- net CHEER in: now also U18.8 (PA0)
- net B'DAY in: now reaches J1.44 (Pin_44)
- net B'DAY in: now also U18.9 (PA1)
- net INTRO in: now reaches J1.45 (Pin_45)
- net INTRO in: now also U18.10 (PA2)
- net SPEC in: now reaches J1.46 (Pin_46)
- net SPEC in: now also U18.11 (PA3)
- net NEXT in: now reaches J1.49 (Pin_49)
- net NEXT in: now also U18.13 (PA5)
- net SKIP in: now reaches J1.51 (Pin_51)
- net SKIP in: now also U18.14 (PA6)
- net AGC 2: now reaches J1.55 (Pin_55)
- net AGC 2: now also U19.13 (PA5)
- net AUDIO IN renamed RESET out
- net RESET out: now also U6.12; no longer J1.120 (Pin_120)
- net DATA OUT renamed CHEER out
- net CHEER out: now also U13.4
- net F.F. renamed AGC 8
- net AGC 8: now also U19.15 (PA7)
- net PLAY: no longer names the net of J1.52 (Pin_52)
- net R.W. renamed DIAG in
- net DIAG in: now also U18.12 (PA4)
- net STOP renamed B'DAY out
- net B'DAY out: now also U12.12
- net /HOLD  renamed /HOLD in
- net /HOLD in: now also R37.2, U6.1
- new net: DS6.2 (A), RP1.10 (R7.2)
- new net: DS5.2 (A), RP1.11 (R6.2)
- new net: DS4.2 (A), RP1.12 (R5.2)
- new net: DS3.2 (A), RP1.13 (R4.2)
- new net: DS2.2 (A), RP1.14 (R3.2)
- new net: DS3.2 (A), RP1.15 (R2.2)
- new net: DS2.2 (A), RP1.16 (R1.2)
- new net: DS7.2 (A), RP1.9 (R8.2)
- new net: R37.2, U25.38 (SO), U25.6 (~{NMI})
- new net: DS6.1 (K), U8.10
- new net: U19.23 (PB1), U8.11
- new net: U14.1 (0), U15.12 (A3), U16.1 (~{CS}), U17.1 (~{CS})
- new net: U16.15 (IN/~{OUT}), U17.15 (IN/~{OUT}), U9.8
- new net: DS4.1 (K), U13.12
- new net: U10.11, U11.12 (A3)
- new net: U10.3, U11.13 (A2)
- new net: DS5.1 (K), U8.8
- new net: R37.1, U6.10, U6.9, Y1.1
- new net: C2.1, CR1.1 (K), CR2.2 (A), R37.2, U25.37 (00), Y1.2
- new net: U19.37 (~{CS2}), U9.3, U9.4
- new net: U19.18 (PB5), U8.5
- new net: DS2.1 (K), U8.6
- new net: C2.2, U25.39 (02), U6.11
- new net: U13.5, U18.16 (PB7)
- new net: U9.6, U9.9
- new net: CR4.2 (A), RP2.1 (R1.1), U25.33 (D0), XU1.1 (R1.1)
- new net: RP2.2 (R2.1), U25.32 (D1), XU1.2 (R2.1)
- new net: CR5.2 (A), RP2.3 (R3.1), U25.31 (D2), XU1.3 (R3.1)
- new net: RP2.4 (R4.1), U25.30 (D3), XU1.4 (R4.1)
- new net: CR6.2 (A), RP2.5 (R5.1), U25.29 (D4), XU1.5 (R5.1)
- new net: RP2.6 (R6.1), U25.28 (D5), XU1.6 (R6.1)
- new net: RP2.7 (R7.1), U25.27 (D6), XU1.7 (R7.1)
- new net: RP2.8 (R8.1), U25.26 (D7), XU1.8 (R8.1)
- new net: U12.13, U18.23 (PB1)
- new net: U23.1 (OEa), U23.15 (OEb), U24.1 (OEa), U24.15 (OEb), U5.1 (OEa), U5.15 (OEb), U6.2
- new net: R37.2, TP2.1, U18.38 (CS1)
- new net: C21.1, CR3.2 (A), R37.2, R37.2, U6.3
- new net: U6.4, U6.5
- new net: DS7.1 (K), U8.12
- new net: DS2.1 (K), U8.2
- new net: U12.11, U18.22 (PB2)
- new net: R37.2, TP2.1, U19.38 (CS1)
- new net: U12.5, U18.19 (PB4)
- new net: U18.37 (~{CS2}), U9.11, U9.5
- new net: U12.9, U18.21 (PB3)
- new net: DS3.1 (K), U8.4
- new net: U13.13, U19.21 (PB3)
- new net: U19.22 (PB2), U8.9
- new net: U13.3, U18.24 (PB0)
- new net: U19.16 (PB7), U8.1
- new net: U13.1, U19.19 (PB4)
- new net: DS3.1 (K), U13.2
- new net: U19.9 (PA1), U6.13
- new net: U12.1, U18.17 (PB6)
- new net: U12.3, U18.18 (PB5)
- new net: U19.17 (PB6), U8.3
- new net: U19.24 (PB0), U8.13
- new net BA0: J1.75 (Pin_75), U18.7 (A0), U19.7 (A0), U20.8 (A0), U21.8 (A0), U22.8 (A0), U24.11 (O5b)
- new net BA1: J1.15 (Pin_15), U18.6 (A1), U19.6 (A1), U20.7 (A1), U21.7 (A1), U22.7 (A1), U24.5 (O2a)
- new net BA10: J1.30 (Pin_30), U14.15 (A0), U24.7 (O3a)
- new net BA11: J1.91 (Pin_91), U14.14 (A1), U24.9 (O4a)
- new net BA12: J1.31 (Pin_31), U14.13 (A2), U5.11 (O5b)
- new net BA2: J1.76 (Pin_76), U11.15 (A0), U18.5 (A2), U19.5 (A2), U20.6 (A2), U21.6 (A2), U22.6 (A2), U24.13 (O6b)
- new net BA3: J1.16 (Pin_16), U11.14 (A1), U18.4 (A3), U19.4 (A3), U20.5 (A3), U21.5 (A3), U22.5 (A3), U24.3 (O1a)
- new net BA4: J1.27 (Pin_27), U10.1, U18.3 (A4), U19.3 (A4), U20.4 (A4), U21.4 (A4), U22.4 (A4), U23.9 (O4a)
- new net BA5: J1.88 (Pin_88), U10.12, U18.2 (A5), U19.2 (A5), U20.3 (A5), U21.3 (A5), U22.3 (A5), U23.7 (O3a)
- new net BA6: J1.28 (Pin_28), U18.40 (CA1), U19.40 (CA1), U20.2 (A6), U21.2 (A6), U22.2 (A6), U23.5 (O2a)
- new net BA7: J1.89 (Pin_89), U15.15 (A0), U20.1 (A7), U21.1 (A7), U22.1 (A7), U23.3 (O1a)
- new net BA8: J1.29, U15.14 (A1), U20.23 (A8), U21.23 (A8), U22.23 (A8), U23.13 (O6b)
- new net BA9: J1.90 (Pin_90), U15.13 (A2), U20.22 (A9), U21.22 (A9), U22.22 (A9), U23.11 (O5b)
- new net DB0: J1.10 (Pin_10), U17.10 (DB2)
- new net DB1: J1.71 (Pin_71), U17.13 (DB3)
- new net DB2: J1.11 (Pin_11), U17.3 (DB0)
- new net DB3: J1.72 (Pin_72), U17.6 (DB1)
- new net DB4: J1.12 (Pin_12), U16.10 (DB2)
- new net DB5: J1.73 (Pin_73), U16.13 (DB3)
- new net DB6: J1.13 (Pin_13), U16.3 (DB0)
- new net DB7: J1.74 (Pin_74), U16.6 (DB1)
- new net SKIP out: J1.120 (Pin_120), U12.2
- new net cpu R/~{W}: U25.34 (R/~{W}), U5.14 (I6)
- new net /CARDS: U10.13, U10.2, U15.2 (1)
- new net /CS U20: U14.9 (7), U20.20 (~{CS})
- new net /CS U21: U14.7 (6), U21.20 (~{CS})
- new net /CS U22: U14.6 (5), U22.20 (~{CS})
- new net /IRQ out: J1.36 (Pin_36), W1.2 (Pin_2)
- new net /RAM: U15.1 (0), U18.36 (/RS), U9.12
- new net /STACK: U15.4 (3), U19.36 (/RS), U9.1
- new net /U18: U15.5 (4), U9.13
- new net /U19: U15.6 (5), U9.2
- no-connect marks 24 -> 126
Other:
- note added: "16v"
- note removed: "checked"
- note removed: "redefine for CPU card slot"
- moved on the sheet: C21, C34, J1, TP2, U7

Commit message: continued routing
Connections:
- net RESET out: now also U13.8; no longer U6.12
- net at U6.13: no longer U19.9 (PA1)
- net at U13.9: now also U19.9 (PA1)
- net at U18.18 (PB5): now also U12.3
- no-connect marks 126 -> 124
Other:
- moved on the sheet: U13D
Changed lines of the file:
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@@
   (no_connect (at 173.355 203.835))
   (no_connect (at 44.45 154.94))
-  (no_connect (at 218.44 16.51))
   (no_connect (at 170.815 193.675))
   (no_connect (at 31.75 25.4))
@@
   (no_connect (at 31.75 127))
   (no_connect (at 157.48 145.415))
-  (no_connect (at 203.2 16.51))
   (no_connect (at 189.23 24.765))
   (no_connect (at 259.715 204.47))
@@
     )
   )
+  (symbol (lib_id "74xx:74LS14") (at 227.965 0.635 0) (unit 6)
+    (in_bom yes) (on_board yes) (dnp no) (fields_autoplaced)
+    (property "Reference" "U6" (at 227.965 -6.1849 0)
+      (effects (font (size 1.27 1.27)))
+    )
+    (property "Value" "7414" (at 227.965 -4.2639 0)
+      (effects (font (size 1.27 1.27)))
+    )
+    (property "Footprint" "Package_DIP:DIP-14_W7.62mm" (at 227.965 0.635 0)
+      (effects (font (size 1.27 1.27)) hide)
+    )
+    (property "Datasheet" "http://www.ti.com/lit/gpn/sn74LS14" (at 227.965 0.635 0)
+      (effects (font (size 1.27 1.27)) hide)
+    )
+    (pin "1")
+    (pin "2")
+    (pin "3")
+    (pin "4")
+    (pin "5")
+    (pin "6")
+    (pin "8")
+    (pin "9")
+    (pin "10")
+    (pin "11")
+    (pin "12")
+    (pin "13")
+    (pin "14")
+    (pin "7")
+    (instances
+      (project "CPU board 0001 rev.a"
+        (path "/972f3ffb-6bde-4480-8d3a-f1aadeb0cbf8"
+          (reference "U6") (unit 6)
+        )
+      )
+    )
+  )
   (symbol (lib_id "power:+5V") (at 277.495 104.775 0) (unit 1)
     (in_bom yes) (on_board yes) (dnp no) (fields_autoplaced)
@@
     )
   )
-  (symbol (lib_id "74xx:74LS14") (at 426.72 137.16 0) (unit 6)
-    (in_bom yes) (on_board yes) (dnp no) (fields_autoplaced)
-    (property "Reference" "U6" (at 426.72 130.3401 0)
-      (effects (font (size 1.27 1.27)))
-    )
-    (property "Value" "7414" (at 426.72 132.2611 0)
-      (effects (font (size 1.27 1.27)))
-    )
-    (property "Footprint" "Package_DIP:DIP-14_W7.62mm" (at 426.72 137.16 0)
-      (effects (font (size 1.27 1.27)) hide)
-    )
-    (property "Datasheet" "http://www.ti.com/lit/gpn/sn74LS14" (at 426.72 137.16 0)
-      (effects (font (size 1.27 1.27)) hide)
-    )
-    (pin "1")
-    (pin "2")
-    (pin "3")
-    (pin "4")
-    (pin "5")
-    (pin "6")
-    (pin "8")
-    (pin "9")
-    (pin "10")
-    (pin "11")
-    (pin "12")
-    (pin "13")
-    (pin "14")
-    (pin "7")
-    (instances
-      (project "CPU board 0001 rev.a"
-        (path "/972f3ffb-6bde-4480-8d3a-f1aadeb0cbf8"
-          (reference "U6") (unit 6)
-        )
-      )
-    )
-  )
   (symbol (lib_id "power:+5V") (at 178.435 21.59 0) (unit 1)
     (in_bom yes) (on_board yes) (dnp no) (fields_autoplaced)
@@
     )
   )
-  (symbol (lib_id "74xx:74LS06") (at 210.82 16.51 0) (unit 4)
+  (symbol (lib_id "74xx:74LS06") (at 426.72 137.16 0) (unit 4)
     (in_bom yes) (on_board yes) (dnp no)
-    (property "Reference" "U13" (at 209.55 15.224 0)
+    (property "Reference" "U13" (at 425.45 135.874 0)
       (effects (font (size 1.27 1.27)))
     )
-    (property "Value" "7406" (at 209.55 17.145 0)
+    (property "Value" "7406" (at 425.45 137.795 0)
       (effects (font (size 1.27 1.27)))
     )
-    (property "Footprint" "Package_DIP:DIP-14_W7.62mm" (at 210.82 16.51 0)
+    (property "Footprint" "Package_DIP:DIP-14_W7.62mm" (at 426.72 137.16 0)
       (effects (font (size 1.27 1.27)) hide)
     )
-    (property "Datasheet" "http://www.ti.com/lit/gpn/sn74LS06" (at 210.82 16.51 0)
+    (property "Datasheet" "http://www.ti.com/lit/gpn/sn74LS06" (at 426.72 137.16 0)
       (effects (font (size 1.27 1.27)) hide)
     )

Commit message: finished rev.a layout
Connections:
- net GND: no longer J1.112 (Pin_112), J1.87 (Pin_87)
- net /RESET: no longer J1.50 (Pin_50), R37.1
- net at R37.1, U6.10, U6.9: now also Y1.2; no longer Y1.1
- net at C2.1, CR1.1 (K), CR2.2 (A)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: now also Y1.1; no longer Y1.2
- net at U18.18 (PB5): now also U12.3
- new net /RESET in: J1.50 (Pin_50), R37.1
- no-connect marks 124 -> 126
Other:
- note added: "112 grounded on rev a schematic, not grounded on the rev a pcb"
- note added: "87 grounded on rev a schematic, not grounded on the rev a pcb"
Changed lines of the file:
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@@
   (junction (at 140.335 66.04) (diameter 0) (color 0 0 0 0)
   )
-  (junction (at 19.05 152.4) (diameter 0) (color 0 0 0 0)
-  )
   (junction (at 80.01 66.04) (diameter 0) (color 0 0 0 0)
   )
@@
   (junction (at 140.335 58.42) (diameter 0) (color 0 0 0 0)
   )
-  (junction (at 19.05 88.9) (diameter 0) (color 0 0 0 0)
-  )
   (junction (at 69.215 58.42) (diameter 0) (color 0 0 0 0)
   )
@@
   (no_connect (at 204.47 31.75))
   (no_connect (at 419.1 98.425))
+  (no_connect (at 31.75 88.9))
   (no_connect (at 183.515 203.835))
   (no_connect (at 267.335 204.47))
@@
   (no_connect (at 257.175 204.47))
   (no_connect (at 269.875 194.31))
+  (no_connect (at 31.75 152.4))
   (no_connect (at 44.45 142.24))
   (no_connect (at 168.275 203.835))
@@
     (stroke (width 0) (type default))
   )
-  (wire (pts (xy 19.05 149.86) (xy 19.05 152.4))
+  (wire (pts (xy 19.05 149.86) (xy 19.05 166.37))
     (stroke (width 0) (type default))
   )
@@
     (stroke (width 0) (type default))
   )
-  (wire (pts (xy 19.05 152.4) (xy 19.05 166.37))
-    (stroke (width 0) (type default))
-  )
   (wire (pts (xy 187.325 95.885) (xy 176.53 95.885))
     (stroke (width 0) (type default))
@@
     (stroke (width 0) (type default))
   )
-  (wire (pts (xy 19.05 45.72) (xy 19.05 88.9))
+  (wire (pts (xy 19.05 45.72) (xy 19.05 106.68))
     (stroke (width 0) (type default))
   )
@@
     (stroke (width 0) (type default))
   )
-  (wire (pts (xy 31.75 88.9) (xy 19.05 88.9))
-    (stroke (width 0) (type default))
-  )
   (wire (pts (xy 88.9 101.6) (xy 85.725 101.6))
     (stroke (width 0) (type default))
@@
     (stroke (width 0) (type default))
   )
-  (wire (pts (xy 31.75 152.4) (xy 19.05 152.4))
-    (stroke (width 0) (type default))
-  )
   (wire (pts (xy 464.185 133.35) (xy 461.645 133.35))
     (stroke (width 0) (type default))
@@
     (stroke (width 0) (type default))
   )
-  (wire (pts (xy 19.05 88.9) (xy 19.05 106.68))
-    (stroke (width 0) (type default))
-  )
   (wire (pts (xy 181.61 72.39) (xy 184.15 72.39))
     (stroke (width 0) (type default))
   )
+  (text "112 grounded on rev a schematic, not grounded on the rev a pcb"
+    (at -47.625 152.4 0)
+    (effects (font (size 1.27 1.27)) (justify left bottom))
+  )
+  (text "87 grounded on rev a schematic, not grounded on the rev a pcb"
+    (at -46.99 89.535 0)
+    (effects (font (size 1.27 1.27)) (justify left bottom))
+  )
   (text "16v" (at 80.01 161.925 0)
     (effects (font (size 1.27 1.27)) (justify left bottom))
@@
     )
   )
-  (global_label "{slash}RESET" (shape input) (at 44.45 149.86 0) (fields_autoplaced)
+  (global_label "{slash}RESET in" (shape input) (at 44.45 149.86 0) (fields_autoplaced)
     (effects (font (size 1.27 1.27)) (justify left))
-    (property "Intersheetrefs" "${INTERSHEET_REFS}" (at 54.4314 149.86 0)
+    (property "Intersheetrefs" "${INTERSHEET_REFS}" (at 57.1528 149.86 0)
       (effects (font (size 1.27 1.27)) (justify left) hide)
     )
@@
     )
   )
-  (global_label "{slash}RESET" (shape input) (at 76.835 154.94 180) (fields_autoplaced)
+  (global_label "{slash}RESET in" (shape input) (at 76.835 154.94 180) (fields_autoplaced)
     (effects (font (size 1.27 1.27)) (justify right))
-    (property "Intersheetrefs" "${INTERSHEET_REFS}" (at 66.8536 154.94 0)
+    (property "Intersheetrefs" "${INTERSHEET_REFS}" (at 64.1322 154.94 0)
       (effects (font (size 1.27 1.27)) (justify right) hide)
     )
@@
     )
   )
-  (symbol (lib_id "Device:Crystal") (at 92.71 101.6 0) (unit 1)
-    (in_bom yes) (on_board yes) (dnp no) (fields_autoplaced)
+  (symbol (lib_id "Device:Crystal") (at 92.71 101.6 0) (mirror y) (unit 1)
+    (in_bom yes) (on_board yes) (dnp no)
     (property "Reference" "Y1" (at 92.71 96.0247 0)
       (effects (font (size 1.27 1.27)))

Commit message: Fix spelling errors with Transport
Connections:
- net at U18.18 (PB5): now also U12.3
