File: Boards/Transport board 0020 rev.1982/Transport board 0020 rev.1982.kicad_sch (KiCad schematic)
At the start: 81 parts, among them J1 CEC card edge connector large, U1 6821, U1 TR1602, U10 LM311, U11 LM741, U12 LM311, U3 DM8602N, U4 7410, U4 ULN2003A, U5 74LS74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

Commit message: Fix spelling errors with Transport
Parts:
- removed C34: 10nF, Capacitor_THT:C_Rect_L7.2mm_W2.5mm_P5.00mm_FKS2_FKP2_MKS2_MKP2, symbol Device:C
- removed RP1 (x2): Spare, Package_DIP:DIP-16_W7.62mm, symbol Device:R_Pack08
- removed U6: 74161, Package_DIP:DIP-16_W7.62mm, symbol 74xx:74LS161
- removed U8: Unused DIP, Package_DIP:DIP-14_W7.62mm, symbol Device:R_Pack07
- added C34: 10nF, Capacitor_THT:C_Rect_L9.0mm_W2.5mm_P7.50mm_MKT, symbol Device:C
- added C34: 100nF, Capacitor_THT:C_Rect_L9.0mm_W2.5mm_P7.50mm_MKT, symbol Device:C
- added C4: 100nF, Capacitor_THT:C_Disc_D3.0mm_W1.6mm_P2.50mm, symbol Device:C
- added R37: 2.2K, Resistor_THT:R_Axial_DIN0309_L9.0mm_D3.2mm_P12.70mm_Horizontal, symbol Device:R
- added U7: AH5012, Package_DIP:DIP-16_W7.62mm, symbol Evan's parts:AH5012
- added U8: 74LS00, symbol 74xx:74LS00
- C21: footprint Capacitor_THT:CP_Radial_Tantal_D4.5mm_P2.50mm -> Evan's parts:CP_Radial_Tantal_D4mm_P3.81mm
- C34: footprint Capacitor_THT:C_Rect_L7.2mm_W2.5mm_P5.00mm_FKS2_FKP2_MKS2_MKP2 -> Capacitor_THT:C_Rect_L9.0mm_W2.5mm_P7.50mm_MKT
- C34: value 39nF -> 20nF; footprint Capacitor_THT:CP_Axial_L11.0mm_D6.0mm_P18.00mm_Horizontal -> Capacitor_THT:C_Rect_L9.0mm_W2.5mm_P7.50mm_MKT
- C4: footprint Capacitor_THT:C_Rect_L7.2mm_W2.5mm_P5.00mm_FKS2_FKP2_MKS2_MKP2 -> Capacitor_THT:C_Disc_D3.0mm_W1.6mm_P2.50mm
- C7: footprint Capacitor_THT:C_Axial_L3.8mm_D2.6mm_P12.50mm_Horizontal -> Capacitor_THT:C_Rect_L7.0mm_W2.5mm_P5.00mm
- TP7: value bits -> ones?
- TP7: value zero crossings -> pulses
- TP7: value carrier detect -> zeroes?
- U10, U11, U12: footprint Package_DIP:DIP-8_W7.62mm -> (none)
- U3, U7: footprint Package_DIP:DIP-16_W7.62mm -> (none)
- U4, U5: footprint Package_DIP:DIP-14_W7.62mm -> (none)
Connections:
- net +12V: now also R37.1, C4.1
- net +5V: now also C34.1, U8.14 (VCC)
- net -12V: now also C34.1; no longer R37.1
- net BCLK: now also J1.62 (Pin_62); no longer U4.9
- net DATA OUT: now also U8.11; no longer U1.25 (TO)
- net F.F.: now also U7.15
- net GND: now also C34.2, C34.2, C4.2, U7.1, U7.16, U8.7 (GND)
- net PB3: now also U8.1, U8.10, U8.2
- net R.W.: now also U7.2
- net at U4.7 (I7), U5.8 (~{Q}): now also U8.5; no longer U1.20 (RI)
- net at TP7.1, U3.11 (A), U4.1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: now also U4.5, U7.9 (~{Q})
- net at U10.6 (STRB): now also C4.1; no longer C4.1
- net at C7.2, R37.1, R37.2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: now also R37.1
- net at C21.1: no longer R37.2
- net at U12.6 (STRB): now also C4.1; no longer C4.1
- new net: U8.3, U8.4
- new net: R37.2, U7.14, U7.3
- new net: U8.12, U8.8
- new net: U1.25 (TO), U8.9
- new net: U8.13, U8.6
- no-connect marks 125 -> 94
Other:
- note added: "9600 Baud"
- note removed: "guess"
- note removed: "there seems to be a duplicate of C10 here on the paper schematic"
- moved on the sheet: C21, C4, U4C
