File: Boards/Transport board 0020 rev.b/Transport board 0020 rev.b.kicad_sch (KiCad schematic)
At the start: 82 parts, among them J1 CEC card edge connector large, U1 6821, U1 TR1602, U10 LM311, U11 LM741, U12 LM311, U3 DM8602N, U4 7410, U4 ULN2003A, U5 74LS74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

Commit message: Fix spelling errors with Transport
Parts:
- removed C34: 10nF, Capacitor_THT:C_Rect_L9.0mm_W2.5mm_P7.50mm_MKT, symbol Device:C
- removed C34: 100nF, Capacitor_THT:C_Rect_L9.0mm_W2.5mm_P7.50mm_MKT, symbol Device:C
- removed C4: 100nF, Capacitor_THT:C_Disc_D3.0mm_W1.6mm_P2.50mm, symbol Device:C
- removed R37: 2.2K, Resistor_THT:R_Axial_DIN0309_L9.0mm_D3.2mm_P12.70mm_Horizontal, symbol Device:R
- removed U7: AH5012, Package_DIP:DIP-16_W7.62mm, symbol Evan's parts:AH5012
- removed U8: 74LS00, symbol 74xx:74LS00
- added C34: 10nF, Capacitor_THT:C_Rect_L7.2mm_W2.5mm_P5.00mm_FKS2_FKP2_MKS2_MKP2, symbol Device:C
- added RP1 (x2): Spare, Package_DIP:DIP-16_W7.62mm, symbol Device:R_Pack08
- added U6: 74161, Package_DIP:DIP-16_W7.62mm, symbol 74xx:74LS161
- added U8: Unused DIP, Package_DIP:DIP-14_W7.62mm, symbol Device:R_Pack07
- C21: footprint Evan's parts:CP_Radial_Tantal_D4mm_P3.81mm -> Capacitor_THT:CP_Radial_Tantal_D4.5mm_P2.50mm
- C34: footprint Capacitor_THT:C_Rect_L9.0mm_W2.5mm_P7.50mm_MKT -> Capacitor_THT:C_Rect_L7.2mm_W2.5mm_P5.00mm_FKS2_FKP2_MKS2_MKP2
- C34: value 20nF -> 39nF; footprint Capacitor_THT:C_Rect_L9.0mm_W2.5mm_P7.50mm_MKT -> Capacitor_THT:CP_Axial_L11.0mm_D6.0mm_P18.00mm_Horizontal
- C4: footprint Capacitor_THT:C_Disc_D3.0mm_W1.6mm_P2.50mm -> Capacitor_THT:C_Rect_L7.2mm_W2.5mm_P5.00mm_FKS2_FKP2_MKS2_MKP2
- C7: footprint Capacitor_THT:C_Rect_L7.0mm_W2.5mm_P5.00mm -> Capacitor_THT:C_Axial_L3.8mm_D2.6mm_P12.50mm_Horizontal
- TP7: value ones? -> bits
- TP7: value pulses -> zero crossings
- TP7: value zeroes? -> carrier detect
- U10, U11, U12: footprint (none) -> Package_DIP:DIP-8_W7.62mm
- U3, U7: footprint (none) -> Package_DIP:DIP-16_W7.62mm
- U4, U5: footprint (none) -> Package_DIP:DIP-14_W7.62mm
Connections:
- net +12V: no longer R37.1
- net +5V: now also C34.1, U6.16 (VCC), U8.14 (R1.2)
- net -12V: now also R37.1
- net BCLK: now also U4.9, U6.11 (Q3); no longer J1.62 (Pin_62)
- net DATA OUT: now also U1.25 (TO)
- net GND: now also C34.2, U6.3 (D0), U6.5 (D2), U6.6 (D3), U6.8 (GND), U8.7 (R7.1)
- net PHI2: now also U6.2 (CP)
- net pup: now also U6.1 (~{MR}), U6.10 (CET), U6.4 (D1), U6.7 (CEP)
- net at U4.7 (I7), U5.8 (~{Q}): now also U1.20 (RI)
- net at TP7.1, U3.11 (A), U4.1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: no longer U4.5, U7.9 (~{Q})
- net at U10.6 (STRB): now also C4.1; no longer C4.1
- net at U12.6 (STRB): now also C4.1; no longer C4.1
- net at C21.1: now also R37.2
- net at U4.10: now also U6.12 (Q2)
- net at U4.11: now also U6.13 (Q1)
- net at U4.8: now also U6.9 (~{PE})
- new net: U4.5, U7.9 (~{Q})
- no-connect marks 94 -> 125
Other:
- note added: "guess"
- note added: "there seems to be a duplicate of C10 here on the paper schematic"
- note removed: "9600 Baud"
- moved on the sheet: C21, C4, U4C
