File: Boards/CPU board 0001 rev.c/CPU board 0001 rev.c.kicad_sch (KiCad schematic)
At the start: 78 parts, among them J1 CEC card edge connector large, U10 7432, U11 7442, U12 7406, U13 7406, U14 7442, U15 7442, U16 M8216, U17 M8216, U18 6532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

Commit message: updated boards per real one
Connections:
- net at U18.18 (PB5): now also U12.3
Other:
- note added: "112 grounded on rev c schematic, not grounded on the rev c pcb"
- note added: "87 grounded on rev c schematic, not grounded on the rev c pcb"
- note removed: "112 grounded on rev a schematic, not grounded on the rev a pcb"
- note removed: "87 grounded on rev a schematic, not grounded on the rev a pcb"
- moved on the sheet: U6F

Commit message: revisions from real life boards
tip130a is actually tip30a, widened holes for crystal, widened holes for big power resistor, fixed cpu board LED resistors
Parts:
- RP1: value 10K -> 330
Connections:
- net at U18.18 (PB5): now also U12.3
Changed lines of the file:
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@@
       (effects (font (size 1.27 1.27)) (justify left))
     )
-    (property "Value" "10K" (at 485.14 139.7 0)
+    (property "Value" "330" (at 485.14 139.7 0)
       (effects (font (size 1.27 1.27)) (justify left))
     )
