File: Boards/Character board 0034 rev.d/Character board 0034 rev.d.kicad_pcb (KiCad board)
At the start: 2 copper layers, 166.4 x 186.7 mm, 40 parts, among them J1 card edge, J2 character connector, J3 power jumper, J4 return jumper, Q1 TIP130A, U1 2.2K, U11 ULN2003A, U12 ULN2003A, U13 7406, U2 2.2K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

Commit message: added logos
Parts:
- added G***: LOGO, Evan's parts:pizza logo, F.Cu at (143.5, 13.3)

Commit message: revisions from real life boards
tip130a is actually tip30a, widened holes for crystal, widened holes for big power resistor, fixed cpu board LED resistors
Parts:
- Q1: value TIP130A -> TIP30A
Changed lines of the file:
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@@
     (fp_line (start 20.32 0) (end 14.66 0)
       (stroke (width 0.1) (type solid)) (layer "F.Fab"))
-    (pad "1" thru_hole circle (at 0 0 270) (size 1.6 1.6) (drill 0.8) (layers "*.Cu" "*.Mask")
+    (pad "1" thru_hole circle (at 0 0 270) (size 2 2) (drill 1) (layers "*.Cu" "*.Mask")
       (net 24 "Net-(Q1-B)") (pintype "passive"))
-    (pad "2" thru_hole oval (at 20.32 0 270) (size 1.6 1.6) (drill 0.8) (layers "*.Cu" "*.Mask")
+    (pad "2" thru_hole circle (at 20.32 0 270) (size 2 2) (drill 1) (layers "*.Cu" "*.Mask")
       (net 92 "Net-(C11-Pad1)") (pintype "passive"))
     (model "${KICAD6_3DMODEL_DIR}/Resistor_THT.3dshapes/R_Axial_DIN0309_L9.0mm_D3.2mm_P20.32mm_Horizontal.wrl"
@@
         (effects (font (size 1 1) (thickness 0.15)))
     )
-    (fp_text value "TIP130A" (at 2.54 -9.435) (layer "F.SilkS")
-        (effects (font (size 1 1) (thickness 0.15)))
-    )
+    (fp_text value "TIP30A" (at 2.54 -9.435) (layer "F.SilkS")
+        (effects (font (size 1 1) (thickness 0.15)))
+    )

Commit message: revised value of resistor to 1k per board
Parts:
- R1: value 100 -> 1K
Changed lines of the file:
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@@
         (effects (font (size 1 1) (thickness 0.15)))
     )
-    (fp_text value "100" (at 10.16 0 90) (layer "F.SilkS")
+    (fp_text value "1K" (at 10.16 0 90) (layer "F.SilkS")
         (effects (font (size 1 1) (thickness 0.15)))
     )
