File: Boards/Character board 0004 rev.b/Character board 0004 rev.b.kicad_sch (KiCad schematic)
At the start: 64 parts, among them J1 card edge, J2 character connector, Q1 2N6125, U1 2.2K, U1 6821, U13 7406, U14 74LS42, U15 LM741, U16 AH5012, U2 2.2K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

Commit message: revised PCBs based on Jen's boards, added rev.c
Parts:
- F1: value 1A -> 3/4A
Connections:
- net A4out: now also DS1.1 (K); no longer DS1.1 (K)
- net A6out: now also DS1.1 (K); no longer DS1.1 (K)
