File: Boards/Solenoid board 0005 rev.b/Solenoid board 0005 rev.b.kicad_pcb (KiCad board)
At the start: 2 copper layers, 190.6 x 177.9 mm, 8 parts, among them J1 character connector, J2 Conn_Coaxial, K1 DIP relay, T1 Transformer_SP_2S

Commit message: layout of solenoid board done
Parts:
- added G***: LOGO, Evan's parts:PTT white_2, F.Cu at (93.8, 18.3)
- moved TB1 356.2 mm to (14.0, 160.7), turned to 90 degrees
- moved K1 282.4 mm to (148.6, 141.2)
- moved TP2 268.5 mm to (155.7, 162.2)
- moved T1 265.6 mm to (121.4, 140.4)
- moved TP1 181.3 mm to (52.2, 171.1)
- moved TB2 176.2 mm to (176.4, 160.7), turned to 90 degrees
- moved J2 60.8 mm to (139.8, 165.1)
- moved J1 52.6 mm to (110.6, 166.4)
Routing:
- net +24VDC: track 0.00 -> 659.5 mm
- net SC6: track 0.00 -> 181.2 mm, vias 0 -> 1
- net CC8: track 0.00 -> 178.8 mm
- net SC5: track 0.00 -> 165.5 mm, vias 0 -> 1
- net CC7: track 0.00 -> 162.3 mm
- net SC4: track 0.00 -> 145.7 mm
- net SC2: track 0.00 -> 145.0 mm
- net SC3: track 0.00 -> 139.9 mm
- net CC6: track 0.00 -> 139.7 mm
- net SC1: track 0.00 -> 125.4 mm
- net CC5: track 0.00 -> 123.3 mm
- net 24R: track 0.00 -> 117.1 mm
- net LC2: track 0.00 -> 112.8 mm
- net CC4: track 0.00 -> 110.8 mm
- net CC3: track 0.00 -> 104.7 mm
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- added copper zone on B.Cu, net +24VDC
- added copper zone on B.Cu, net SIGNAL GND.
Other:
- outline, holes or cut-outs redrawn
- board text added: "1"
- board text added: "10"
- board text added: "11"
- board text added: "12"
- board text added: "13"
- board text added: "14"
- board text added: "15"
- board text added: "16"
- board text added: "2"
- board text added: "25"
- board text added: "26"
- board text added: "3"
- board text added: "4"
- board text added: "5"
- board text added: "6"
- board text added: "7"
- board text added: "8"
- board text added: "9"
- board text added: "Conn_01x16_Pin"
- board text added: "J1"
- board text added: "J2"
- board text added: "K1"
- board text added: "L1"
- board text added: "L2"
- board text added: "L3"
- board text added: "L4"
- board text added: "L5"
- board text added: "L6"
- board text added: "L7"
- board text added: "L8"
- board text added: "PART 07-0005 REV B"
- board text added: "SJC4A/94VO/2-82"
- board text added: "SOLENOID BD. ASSY 06-0005 REV B"
- board text added: "T1"
- board text added: "TB1"
- board text added: "TB2"
- board text added: "TP1"
- board text added: "TP2"
