File: Adapters/8216 substitute/8216 substitute.kicad_sch (KiCad schematic)
At the start: 3 parts, among them U1 74LS245, U2 M8216, U3 M8216

Commit message: 8216 adapter fab
Parts:
- U1: footprint (none) -> Package_DIP:DIP-20_W7.62mm
- U2, U3: footprint (none) -> Package_DIP:DIP-16_W7.62mm
