File: Boards/CPU board 0001 rev.d/CPU board 0001 rev.d.kicad_sch (KiCad schematic)
At the start: 78 parts, among them J1 CEC card edge connector large, U10 7432, U11 7442, U12 7406, U13 7406, U14 7442, U15 7442, U16 M8216, U17 M8216, U18 6532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

Commit message: updated boards per real one
Connections:
- net +5V: now also U20.24 (VCC), U22.24 (VCC)
- net at U18.18 (PB5): now also U12.3
- no-connect marks 130 -> 128
Other:
- moved on the sheet: U13E, U22, U6F

Commit message: revisions from real life boards
tip130a is actually tip30a, widened holes for crystal, widened holes for big power resistor, fixed cpu board LED resistors
Parts:
- RP1: value 10K -> 330
Connections:
- net at U18.18 (PB5): now also U12.3
Changed lines of the file:
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@@
       (effects (font (size 1.27 1.27)) (justify left))
     )
-    (property "Value" "10K" (at 485.14 139.7 0)
+    (property "Value" "330" (at 485.14 139.7 0)
       (effects (font (size 1.27 1.27)) (justify left))
     )

Commit message: fixed rev.d pull up on CS and added render and schematic
Parts:
- added R10: 1K, Resistor_THT:R_Axial_DIN0309_L9.0mm_D3.2mm_P12.70mm_Horizontal, symbol Device:R
Connections:
- net +5V: now also R10.1
- net /CS 2732: now also R10.2
- net at U18.18 (PB5): now also U12.3
Other:
- moved on the sheet: C2, C21, C34, CR1, CR2, CR3, CR4, CR5, CR6, DS2, DS3, DS4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
