File: Boards/Transport board 0020 rev.d/Transport board 0020 rev.d.kicad_sch (KiCad schematic)
At the start: 83 parts, among them J1 CEC card edge connector large, U1 6821, U1 TR1602, U10 LM311, U11 LM741, U12 LM311, U3 DM8602N, U4 7410, U4 ULN2003A, U5 74LS74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

Commit message: added lights DE9 adapter
Parts:
- renumbered C34 to C1, C4 to C10, C7 to C11, C34 to C12, C21 to C13, C21 to C14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
