File: Boards/LCD board modified/LCD board modified.kicad_pcb (KiCad board)
At the start: 2 copper layers, 151.9 x 80.6 mm, 19 parts, among them Q1 2N2222A, SW1 RESET, SW2 ENTER, SW3 DOWN, SW4 UP

Commit message: transport board silk update
Parts:
- added G***: LOGO, Evan's parts:Evan Logo, F.Cu at (78.5, 43.5)
Other:
- board text added: "cyberamic control center HC11 display/comtrol board"

Commit message: fixed typo
Other:
- board text added: "cyberamic control center HC11 display/control board"
- board text removed: "cyberamic control center HC11 display/comtrol board"
Changed lines of the file:
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@@
 			(psa4output no)
 			(plot_black_and_white yes)
-			(plotinvisibletext no)
 			(sketchpadsonfab no)
 			(plotpadnumbers no)
@@
 		)
 	)
-	(gr_text "cyberamic control center HC11 display/comtrol board"
+	(gr_text "cyberamic control center HC11 display/control board"
 		(at 61 33.5 0)
 		(layer "F.SilkS")
